File: pcb/memekbd/memekbd.sch (KiCad schematic (older format))
At the start: 92 parts

Commit message: Add foostan's kicad libraries. Finish design of schematic, passes ERC
Parts:
- added C1, C10, C11, C12, C13, C14, C15, C16, C17, C18, C19, C2, C20, C21, C22, C23, C24, C25, C26, C27, C28, C29, C3, C30, C31, C32, C33, C34, C35, C36, C37, C38, C39, C4, C40, C41, C42, C43, C44, C45, C46, C5, C6, C7, C8, C9: 0.1uF, symbol Device:C_Small
- added J1, J2: AudioJack4, symbol Connector:AudioJack4
- added LED1, LED10, LED11, LED12, LED13, LED14, LED15, LED16, LED17, LED18, LED19, LED2, LED20, LED21, LED22, LED23, LED24, LED25, LED26, LED27, LED28, LED29, LED3, LED30, LED31, LED32, LED33, LED34, LED35, LED36, LED37, LED38, LED39, LED4, LED40, LED41, LED42, LED43, LED44, LED45, LED46, LED5, LED6, LED7, LED8, LED9: YS-SK6812MINI-E, symbol kbd:YS-SK6812MINI-E
- added R1, R2, R3, R4: 10k, symbol Device:R
- added SW47, SW48: SW_Push, symbol Switch:SW_Push
- added U1, U2: ProMicro, symbol kbd:ProMicro
- gave numbers to parts that had none: 92
Connections:
- net lcol0: now also U1.7 (4/D4)
- net lcol1: now also U1.8 (5/C6)
- net lcol2: now also U1.9 (6/D7)
- net lcol3: now also U1.10 (7/E6)
- net lcol4: now also U1.11 (8/B4)
- net lrow0: now also U1.20 (F4/A3)
- net lrow1: now also U1.19 (F5/A2)
- net lrow2: now also U1.18 (F6/A1)
- net lrow3: now also U1.17 (F7/A0)
- net lrow4: now also U1.16 (B1/15)
- net rcol0: now also U2.7 (4/D4)
- net rcol1: now also U2.8 (5/C6)
- net rcol2: now also U2.9 (6/D7)
- net rcol3: now also U2.10 (7/E6)
- net rcol4: now also U2.11 (8/B4)
- net rrow0: now also U2.20 (F4/A3)
- net rrow1: now also U2.19 (F5/A2)
- net rrow2: now also U2.18 (F6/A1)
- net rrow3: now also U2.17 (F7/A0)
- net rrow4: now also U2.16 (B1/15)
- new net: LED10.4 (DIN), LED5.2 (DOUT)
- new net: LED10.2 (DOUT), LED15.4 (DIN)
- new net: LED1.4 (DIN), LED15.2 (DOUT)
- new net: LED1.2 (DOUT), LED6.4 (DIN)
- new net: LED11.4 (DIN), LED6.2 (DOUT)
- new net: LED11.2 (DOUT), LED16.4 (DIN)
- new net: LED16.2 (DOUT), LED20.4 (DIN)
- new net: LED2.4 (DIN), LED20.2 (DOUT)
- new net: LED2.2 (DOUT), LED7.4 (DIN)
- new net: LED12.4 (DIN), LED7.2 (DOUT)
- new net: LED12.2 (DOUT), LED17.4 (DIN)
- new net: LED17.2 (DOUT), LED21.4 (DIN)
- new net: LED21.2 (DOUT), LED3.4 (DIN)
- new net: LED3.2 (DOUT), LED8.4 (DIN)
- new net: LED13.4 (DIN), LED8.2 (DOUT)
- new net: LED13.2 (DOUT), LED18.4 (DIN)
- new net: LED18.2 (DOUT), LED22.4 (DIN)
- new net: LED22.2 (DOUT), LED4.4 (DIN)
- new net: LED4.2 (DOUT), LED9.4 (DIN)
- new net: LED14.4 (DIN), LED9.2 (DOUT)
- new net: LED14.2 (DOUT), LED19.4 (DIN)
- new net: LED19.2 (DOUT), LED23.4 (DIN)
- new net: LED24.2 (DOUT), LED29.4 (DIN)
- new net: LED24.4 (DIN), LED38.2 (DOUT)
- new net: LED29.2 (DOUT), LED34.4 (DIN)
- new net: LED34.2 (DOUT), LED39.4 (DIN)
- new net: LED39.2 (DOUT), LED43.4 (DIN)
- new net: LED25.4 (DIN), LED43.2 (DOUT)
- new net: LED25.2 (DOUT), LED30.4 (DIN)
- new net: LED30.2 (DOUT), LED35.4 (DIN)
- new net: LED35.2 (DOUT), LED40.4 (DIN)
- new net: LED40.2 (DOUT), LED44.4 (DIN)
- new net: LED26.4 (DIN), LED44.2 (DOUT)
- new net: LED26.2 (DOUT), LED31.4 (DIN)
- new net: LED31.2 (DOUT), LED36.4 (DIN)
- new net: LED36.2 (DOUT), LED41.4 (DIN)
- new net: LED41.2 (DOUT), LED45.4 (DIN)
- new net: LED27.4 (DIN), LED45.2 (DOUT)
- new net: LED27.2 (DOUT), LED32.4 (DIN)
- new net: LED32.2 (DOUT), LED37.4 (DIN)
- new net: LED37.2 (DOUT), LED42.4 (DIN)
- new net: LED42.2 (DOUT), LED46.4 (DIN)
- new net: LED28.2 (DOUT), LED33.4 (DIN)
- new net: LED33.2 (DOUT), LED38.4 (DIN)
- new net +5V: C1.1, C10.1, C11.1, C12.1, C13.1, C14.1, C15.1, C16.1, C17.1, C18.1, C19.1, C2.1, C20.1, C21.1, C22.1, C23.1, C24.1, C25.1, C26.1, C27.1, C28.1, C29.1, C3.1, C30.1, C31.1, C32.1, C33.1, C34.1, C35.1, C36.1, C37.1, C38.1, C39.1, C4.1, C40.1, C41.1, C42.1, C43.1, C44.1, C45.1, C46.1, C5.1, C6.1, C7.1, C8.1, C9.1, J1.T, J2.T, LED1.1 (VDD), LED10.1 (VDD), LED11.1 (VDD), LED12.1 (VDD), LED13.1 (VDD), LED14.1 (VDD), LED15.1 (VDD), LED16.1 (VDD), LED17.1 (VDD), LED18.1 (VDD), LED19.1 (VDD), LED2.1 (VDD), LED20.1 (VDD), LED21.1 (VDD), LED22.1 (VDD), LED23.1 (VDD), LED24.1 (VDD), LED25.1 (VDD), LED26.1 (VDD), LED27.1 (VDD), LED28.1 (VDD), LED29.1 (VDD), LED3.1 (VDD), LED30.1 (VDD), LED31.1 (VDD), LED32.1 (VDD), LED33.1 (VDD), LED34.1 (VDD), LED35.1 (VDD), LED36.1 (VDD), LED37.1 (VDD), LED38.1 (VDD), LED39.1 (VDD), LED4.1 (VDD), LED40.1 (VDD), LED41.1 (VDD), LED42.1 (VDD), LED43.1 (VDD), LED44.1 (VDD), LED45.1 (VDD), LED46.1 (VDD), LED5.1 (VDD), LED6.1 (VDD), LED7.1 (VDD), LED8.1 (VDD), LED9.1 (VDD), R1.2, R2.2, R3.2, R4.2, U1.21 (VCC), U2.21 (VCC)
- new net GND: C1.2, C10.2, C11.2, C12.2, C13.2, C14.2, C15.2, C16.2, C17.2, C18.2, C19.2, C2.2, C20.2, C21.2, C22.2, C23.2, C24.2, C25.2, C26.2, C27.2, C28.2, C29.2, C3.2, C30.2, C31.2, C32.2, C33.2, C34.2, C35.2, C36.2, C37.2, C38.2, C39.2, C4.2, C40.2, C41.2, C42.2, C43.2, C44.2, C45.2, C46.2, C5.2, C6.2, C7.2, C8.2, C9.2, J1.S, J2.S, LED1.3 (VSS), LED10.3 (VSS), LED11.3 (VSS), LED12.3 (VSS), LED13.3 (VSS), LED14.3 (VSS), LED15.3 (VSS), LED16.3 (VSS), LED17.3 (VSS), LED18.3 (VSS), LED19.3 (VSS), LED2.3 (VSS), LED20.3 (VSS), LED21.3 (VSS), LED22.3 (VSS), LED23.3 (VSS), LED24.3 (VSS), LED25.3 (VSS), LED26.3 (VSS), LED27.3 (VSS), LED28.3 (VSS), LED29.3 (VSS), LED3.3 (VSS), LED30.3 (VSS), LED31.3 (VSS), LED32.3 (VSS), LED33.3 (VSS), LED34.3 (VSS), LED35.3 (VSS), LED36.3 (VSS), LED37.3 (VSS), LED38.3 (VSS), LED39.3 (VSS), LED4.3 (VSS), LED40.3 (VSS), LED41.3 (VSS), LED42.3 (VSS), LED43.3 (VSS), LED44.3 (VSS), LED45.3 (VSS), LED46.3 (VSS), LED5.3 (VSS), LED6.3 (VSS), LED7.3 (VSS), LED8.3 (VSS), LED9.3 (VSS), SW47.2, SW48.2, U1.23 (GND), U1.3 (GND), U1.4 (GND), U2.23 (GND), U2.3 (GND), U2.4 (GND)
- new net lLED: LED5.4 (DIN), U1.1 (TX0/D3)
- new net lRST: SW47.1, U1.22 (RST)
- new net lSCL: J1.R1, R2.1, U1.6 (3/D0/SCL)
- new net lSDA: J1.R2, R1.1, U1.5 (2/D1/SDA)
- new net rLED: LED28.4 (DIN), U2.1 (TX0/D3)
- new net rRST: SW48.1, U2.22 (RST)
- new net rSCL: J2.R1, R4.1, U2.6 (3/D0/SCL)
- new net rSDA: J2.R2, R3.1, U2.5 (2/D1/SDA)
- no-connect marks 0 -> 14

Commit message: Assign footprints.
Parts:
- C1, C10, C11, C12, C13, C14, C15, C16, C17, C18, C19, C2, C20, C21, C22, C23, C24, C25, C26, C27, C28, C29, C3, C30, C31, C32, C33, C34, C35, C36, C37, C38, C39, C4, C40, C41, C42, C43, C44, C45, C46, C5, C6, C7, C8, C9: footprint (none) -> Capacitor_THT:C_Disc_D6.0mm_W2.5mm_P5.00mm
- J1, J2: footprint (none) -> kbd:MJ-4PP-9_1side
- LED1, LED10, LED11, LED12, LED13, LED14, LED15, LED16, LED17, LED18, LED19, LED2, LED20, LED21, LED22, LED23, LED24, LED25, LED26, LED27, LED28, LED29, LED3, LED30, LED31, LED32, LED33, LED34, LED35, LED36, LED37, LED38, LED39, LED4, LED40, LED41, LED42, LED43, LED44, LED45, LED46, LED5, LED6, LED7, LED8, LED9: footprint (none) -> kbd:YS-SK6812MINI-E
- R1, R2, R3, R4: footprint (none) -> Resistor_THT:R_Axial_DIN0207_L6.3mm_D2.5mm_P7.62mm_Horizontal
- SW1, SW10, SW11, SW12, SW13, SW14, SW15, SW16, SW17, SW18, SW19, SW2, SW20, SW21, SW22, SW23, SW24, SW25, SW26, SW27, SW28, SW29, SW3, SW30, SW31, SW32, SW33, SW34, SW35, SW36, SW37, SW38, SW39, SW4, SW40, SW41, SW42, SW43, SW44, SW45, SW46, SW5, SW6, SW7, SW8, SW9: footprint (none) -> kbd:CherryMX_Hotswap
- SW47, SW48: footprint (none) -> Button_Switch_THT:SW_PUSH_6mm_H7.3mm
- U1, U2: footprint (none) -> kbd:ProMicro_v3.5

Commit message: Most of pcb layout work.
Parts:
- removed J1, J2: AudioJack4, kbd:MJ-4PP-9_1side, symbol Connector:AudioJack4
- added J1, J2: MJ-4PP-9, kbd:MJ-4PP-9_1side, symbol kbd:MJ-4PP-9
Connections:
- net +5V: now also J1.B, J2.B
- net GND: now also J1.A, J2.A
- net lSCL: now also J1.C
- net lSDA: now also J1.D
- net rSCL: now also J2.C
- net rSDA: now also J2.D
Other:
- moved on the sheet: R1, R2, R3, R4
Changed lines of the file:
@@
 $EndComp
 $Comp
-L Connector:AudioJack4 J1
-U 1 1 60D94451
-P 15750 3650
-F 0 "J1" H 15707 3975 50  0000 C CNN
-F 1 "AudioJack4" H 15707 3884 50  0000 C CNN
-F 2 "kbd:MJ-4PP-9_1side" H 15750 3650 50  0001 C CNN
-F 3 "~" H 15750 3650 50  0001 C CNN
-	1    15750 3650
-	1    0    0    -1
-$EndComp
-$Comp
-L Connector:AudioJack4 J2
-U 1 1 60D97F5C
-P 18250 3650
-F 0 "J2" H 18207 3975 50  0000 C CNN
-F 1 "AudioJack4" H 18207 3884 50  0000 C CNN
-F 2 "kbd:MJ-4PP-9_1side" H 18250 3650 50  0001 C CNN
-F 3 "~" H 18250 3650 50  0001 C CNN
-	1    18250 3650
-	1    0    0    -1
-$EndComp
-$Comp
 L power:GND #PWR0129
 U 1 1 60D9B008
@@
 L power:GND #PWR0127
 U 1 1 60D9B386
-P 15950 3550
-F 0 "#PWR0127" H 15950 3300 50  0001 C CNN
-F 1 "GND" V 15955 3422 50  0000 R CNN
-F 2 "" H 15950 3550 50  0001 C CNN
-F 3 "" H 15950 3550 50  0001 C CNN
-	1    15950 3550
-	0    -1   -1   0
-$EndComp
-$Comp
-L power:GND #PWR0136
-U 1 1 60D9B90C
-P 18450 3550
-F 0 "#PWR0136" H 18450 3300 50  0001 C CNN
-F 1 "GND" V 18455 3422 50  0000 R CNN
-F 2 "" H 18450 3550 50  0001 C CNN
-F 3 "" H 18450 3550 50  0001 C CNN
-	1    18450 3550
-	0    -1   -1   0
+P 15875 3500
+F 0 "#PWR0127" H 15875 3250 50  0001 C CNN
+F 1 "GND" V 15880 3372 50  0000 R CNN
+F 2 "" H 15875 3500 50  0001 C CNN
+F 3 "" H 15875 3500 50  0001 C CNN
+	1    15875 3500
+	-1   0    0    1
 $EndComp
 $Comp
@@
 L power:+5V #PWR0128
 U 1 1 60D9D453
-P 15950 3850
-F 0 "#PWR0128" H 15950 3700 50  0001 C CNN
-F 1 "+5V" V 15965 3978 50  0000 L CNN
-F 2 "" H 15950 3850 50  0001 C CNN
-F 3 "" H 15950 3850 50  0001 C CNN
-	1    15950 3850
-	0    1    1    0
-$EndComp
-$Comp
-L power:+5V #PWR0137
-U 1 1 60D9DA3D
-P 18450 3850
-F 0 "#PWR0137" H 18450 3700 50  0001 C CNN
-F 1 "+5V" V 18465 3978 50  0000 L CNN
-F 2 "" H 18450 3850 50  0001 C CNN
-F 3 "" H 18450 3850 50  0001 C CNN
-	1    18450 3850
-	0    1    1    0
+P 15875 3875
+F 0 "#PWR0128" H 15875 3725 50  0001 C CNN
+F 1 "+5V" V 15890 4003 50  0000 L CNN
+F 2 "" H 15875 3875 50  0001 C CNN
+F 3 "" H 15875 3875 50  0001 C CNN
+	1    15875 3875
+	-1   0    0    1
 $EndComp
 $Comp
@@
 lSCL
 $Comp
-L Device:R R1
-U 1 1 60DFBED0
-P 16300 3500
-F 0 "R1" H 16230 3454 50  0000 R CNN
-F 1 "10k" H 16230 3545 50  0000 R CNN
-F 2 "Resistor_THT:R_Axial_DIN0207_L6.3mm_D2.5mm_P7.62mm_Horizontal" V 16230 3500 50  0001 C CNN
-F 3 "~" H 16300 3500 50  0001 C CNN
-	1    16300 3500
-	-1   0    0    1
-$EndComp
-$Comp
-L power:+5V #PWR0131
-U 1 1 60DFD705
-P 16300 3350
-F 0 "#PWR0131" H 16300 3200 50  0001 C CNN
-F 1 "+5V" V 16315 3478 50  0000 L CNN
-F 2 "" H 16300 3350 50  0001 C CNN
-F 3 "" H 16300 3350 50  0001 C CNN
-	1    16300 3350
-	1    0    0    -1
-$EndComp
-$Comp
 L Device:R R2
 U 1 1 60E00297
-P 16600 3500
-F 0 "R2" H 16530 3454 50  0000 R CNN
-F 1 "10k" H 16530 3545 50  0000 R CNN
-F 2 "Resistor_THT:R_Axial_DIN0207_L6.3mm_D2.5mm_P7.62mm_Horizontal" V 16530 3500 50  0001 C CNN
-F 3 "~" H 16600 3500 50  0001 C CNN
-	1    16600 3500
+P 16600 3525
+F 0 "R2" H 16530 3479 50  0000 R CNN
+F 1 "10k" H 16530 3570 50  0000 R CNN
+F 2 "Resistor_THT:R_Axial_DIN0207_L6.3mm_D2.5mm_P7.62mm_Horizontal" V 16530 3525 50  0001 C CNN
+F 3 "~" H 16600 3525 50  0001 C CNN
+	1    16600 3525
 	-1   0    0    1
 $EndComp
@@
 L power:+5V #PWR0132
 U 1 1 60E0029D
-P 16600 3350
-F 0 "#PWR0132" H 16600 3200 50  0001 C CNN
-F 1 "+5V" V 16615 3478 50  0000 L CNN
-F 2 "" H 16600 3350 50  0001 C CNN
-F 3 "" H 16600 3350 50  0001 C CNN
-	1    16600 3350
+P 16600 3375
+F 0 "#PWR0132" H 16600 3225 50  0001 C CNN
+F 1 "+5V" V 16615 3503 50  0000 L CNN
+F 2 "" H 16600 3375 50  0001 C CNN
+F 3 "" H 16600 3375 50  0001 C CNN
+	1    16600 3375
 	1    0    0    -1
 $EndComp
 Wire Wire Line
-	16600 3750 16600 3650
+	16600 3725 16600 3675
 Wire Wire Line
-	15950 3750 16600 3750
-Wire Wire Line
-	15950 3650 16300 3650
-Text Label 15950 3650 0    50   ~ 0
+	15750 3725 16600 3725
+Text Label 15750 3675 0    50   ~ 0
 lSDA
-Text Label 15950 3750 0    50   ~ 0
+Text Label 15750 3725 0    50   ~ 0
 lSCL
 Text Label 17800 2250 2    50   ~ 0
@@
 L Device:R R3
 U 1 1 60E5D7AF
-P 18800 3500
-F 0 "R3" H 18730 3454 50  0000 R CNN
-F 1 "10k" H 18730 3545 50  0000 R CNN
-F 2 "Resistor_THT:R_Axial_DIN0207_L6.3mm_D2.5mm_P7.62mm_Horizontal" V 18730 3500 50  0001 C CNN
-F 3 "~" H 18800 3500 50  0001 C CNN
-	1    18800 3500
+P 18525 3475
+F 0 "R3" H 18455 3429 50  0000 R CNN
+F 1 "10k" H 18455 3520 50  0000 R CNN
+F 2 "Resistor_THT:R_Axial_DIN0207_L6.3mm_D2.5mm_P7.62mm_Horizontal" V 18455 3475 50  0001 C CNN
+F 3 "~" H 18525 3475 50  0001 C CNN
+	1    18525 3475
 	-1   0    0    1
 $EndComp
@@
 L power:+5V #PWR0138
 U 1 1 60E5D7B5
-P 18800 3350
-F 0 "#PWR0138" H 18800 3200 50  0001 C CNN
-F 1 "+5V" V 18815 3478 50  0000 L CNN
-F 2 "" H 18800 3350 50  0001 C CNN
-F 3 "" H 18800 3350 50  0001 C CNN
-	1    18800 3350
+P 18525 3325
+F 0 "#PWR0138" H 18525 3175 50  0001 C CNN
+F 1 "+5V" V 18540 3453 50  0000 L CNN
+F 2 "" H 18525 3325 50  0001 C CNN
+F 3 "" H 18525 3325 50  0001 C CNN
+	1    18525 3325
 	1    0    0    -1
 $EndComp
@@
 L Device:R R4
 U 1 1 60E5D7BB
-P 19100 3500
-F 0 "R4" H 19030 3454 50  0000 R CNN
-F 1 "10k" H 19030 3545 50  0000 R CNN
-F 2 "Resistor_THT:R_Axial_DIN0207_L6.3mm_D2.5mm_P7.62mm_Horizontal" V 19030 3500 50  0001 C CNN
-F 3 "~" H 19100 3500 50  0001 C CNN
-	1    19100 3500
+P 18825 3475
+F 0 "R4" H 18755 3429 50  0000 R CNN
+F 1 "10k" H 18755 3520 50  0000 R CNN
+F 2 "Resistor_THT:R_Axial_DIN0207_L6.3mm_D2.5mm_P7.62mm_Horizontal" V 18755 3475 50  0001 C CNN
+F 3 "~" H 18825 3475 50  0001 C CNN
+	1    18825 3475
 	-1   0    0    1
 $EndComp
@@
 L power:+5V #PWR0139
 U 1 1 60E5D7C1
-P 19100 3350
-F 0 "#PWR0139" H 19100 3200 50  0001 C CNN
-F 1 "+5V" V 19115 3478 50  0000 L CNN
-F 2 "" H 19100 3350 50  0001 C CNN
-F 3 "" H 19100 3350 50  0001 C CNN
-	1    19100 3350
+P 18825 3325
+F 0 "#PWR0139" H 18825 3175 50  0001 C CNN
+F 1 "+5V" V 18840 3453 50  0000 L CNN
+F 2 "" H 18825 3325 50  0001 C CNN
+F 3 "" H 18825 3325 50  0001 C CNN
+	1    18825 3325
 	1    0    0    -1
 $EndComp
 Wire Wire Line
-	19100 3750 19100 3650
+	18825 3675 18825 3625
 Wire Wire Line
-	18450 3750 19100 3750
+	18150 3675 18825 3675
 Wire Wire Line
-	18450 3650 18800 3650
-Text Label 18450 3650 0    50   ~ 0
+	18150 3625 18525 3625
+Text Label 18150 3625 0    50   ~ 0
 rSDA
-Text Label 18450 3750 0    50   ~ 0
+Text Label 18150 3675 0    50   ~ 0
 rSCL
 Text Label 2100 7000 2    50   ~ 0
@@
 $EndComp
 NoConn ~ 19200 1850
+$Comp
+L kbd:MJ-4PP-9 J1
+U 1 1 614F36EF
+P 15550 3700
+F 0 "J1" H 15581 3976 50  0000 C CNN
+F 1 "MJ-4PP-9" H 15581 3885 50  0000 C CNN
+F 2 "kbd:MJ-4PP-9_1side" H 15825 3875 50  0001 C CNN
+F 3 "~" H 15825 3875 50  0001 C CNN
+	1    15550 3700
+	1    0    0    -1
+$EndComp
+$Comp
+L kbd:MJ-4PP-9 J2
+U 1 1 614F5099
+P 17950 3650
+F 0 "J2" H 17981 3926 50  0000 C CNN
+F 1 "MJ-4PP-9" H 17981 3835 50  0000 C CNN
+F 2 "kbd:MJ-4PP-9_1side" H 18225 3825 50  0001 C CNN
+F 3 "~" H 18225 3825 50  0001 C CNN
+	1    17950 3650
+	1    0    0    -1
+$EndComp
+Wire Wire Line
+	15750 3625 15875 3625
+Wire Wire Line
+	15875 3625 15875 3500
+Wire Wire Line
+	15750 3775 15875 3775
+Wire Wire Line
+	15875 3775 15875 3875
+Wire Wire Line
+	15750 3675 16300 3675
+$Comp
+L power:+5V #PWR0131
+U 1 1 60DFD705
+P 16300 3375
+F 0 "#PWR0131" H 16300 3225 50  0001 C CNN
+F 1 "+5V" V 16315 3503 50  0000 L CNN
+F 2 "" H 16300 3375 50  0001 C CNN
+F 3 "" H 16300 3375 50  0001 C CNN
+	1    16300 3375
+	1    0    0    -1
+$EndComp
+$Comp
+L Device:R R1
+U 1 1 60DFBED0
+P 16300 3525
+F 0 "R1" H 16230 3479 50  0000 R CNN
+F 1 "10k" H 16230 3570 50  0000 R CNN
+F 2 "Resistor_THT:R_Axial_DIN0207_L6.3mm_D2.5mm_P7.62mm_Horizontal" V 16230 3525 50  0001 C CNN
+F 3 "~" H 16300 3525 50  0001 C CNN
+	1    16300 3525
+	-1   0    0    1
+$EndComp
+$Comp
+L power:+5V #PWR0136
+U 1 1 615CFE82
+P 18275 3825
+F 0 "#PWR0136" H 18275 3675 50  0001 C CNN
+F 1 "+5V" V 18290 3953 50  0000 L CNN
+F 2 "" H 18275 3825 50  0001 C CNN
+F 3 "" H 18275 3825 50  0001 C CNN
+	1    18275 3825
+	-1   0    0    1
+$EndComp
+Wire Wire Line
+	18150 3725 18275 3725
+Wire Wire Line
+	18275 3725 18275 3825
+$Comp
+L power:GND #PWR0137
+U 1 1 615D8D20
+P 18275 3450
+F 0 "#PWR0137" H 18275 3200 50  0001 C CNN
+F 1 "GND" V 18280 3322 50  0000 R CNN
+F 2 "" H 18275 3450 50  0001 C CNN
+F 3 "" H 18275 3450 50  0001 C CNN
+	1    18275 3450
+	-1   0    0    1
+$EndComp
+Wire Wire Line
+	18275 3575 18275 3450
+Wire Wire Line
+	18275 3575 18150 3575
 $EndSCHEMATC
