File: pcb/memekbd.kicad_pcb (KiCad board)
At the start: 2 copper layers, 134.1 x 130.9 mm, 209 parts, among them J1 AudioJack4, J2 AudioJack4, SW1 SW_Push, SW10 SW_Push, SW11 SW_Push, SW12 SW_Push, SW13 SW_Push, SW14 SW_Push, SW15 SW_Push, SW16 SW_Push, SW17 SW_Push, SW18 SW_Push, SW19 SW_Push, SW2 SW_Push, SW20 SW_Push, SW21 SW_Push, SW22 SW_Push, SW23 SW_Push, SW24 SW_Push, SW25 SW_Push, SW26 SW_Push, SW27 SW_Push, SW28 SW_Push, SW29 SW_Push, SW3 SW_Push, SW30 SW_Push, SW31 SW_Push, SW32 SW_Push, SW33 SW_Push, SW34 SW_Push, SW35 SW_Push, SW36 SW_Push, SW37 SW_Push, SW38 SW_Push, SW39 SW_Push, SW4 SW_Push, SW40 SW_Push, SW41 SW_Push, SW42 SW_Push, SW43 SW_Push, SW44 SW_Push, SW45 SW_Push, SW46 SW_Push, SW47 SW_Push, SW48 SW_Push, SW5 SW_Push, SW6 SW_Push, SW7 SW_Push, SW8 SW_Push, SW9 SW_Push, U1 ProMicro, U2 ProMicro

Commit message: Routing progress
Routing:
- net Net-(LED20-Pad2): track 1.52 -> 30.1 mm, vias 1 -> 2

Commit message: Create only mounting hole, edge, and tracks portion
Parts:
- added REF**: MountingHole_5.3mm_M5_ISO7380, MountingHole:MountingHole_5.3mm_M5_ISO7380, B.Cu at (229.2, 257.0)
- added REF**: MountingHole_3.2mm_M3_ISO7380, MountingHole:MountingHole_3.2mm_M3_ISO7380, B.Cu at (318.8, 241.8)
- added REF**: MountingHole_3.2mm_M3_ISO7380, MountingHole:MountingHole_3.2mm_M3_ISO7380, B.Cu at (219.2, 274.5)
- added REF**: MountingHole_3.2mm_M3_ISO7380, MountingHole:MountingHole_3.2mm_M3_ISO7380, B.Cu at (317.2, 210.8)
- added REF**: MountingHole_3.2mm_M3_ISO7380, MountingHole:MountingHole_3.2mm_M3_ISO7380, B.Cu at (261.0, 253.8)
- added REF**: MountingHole_5.3mm_M5_ISO7380, MountingHole:MountingHole_5.3mm_M5_ISO7380, F.Cu at (104.8, 173.2)
- added REF**: MountingHole_5.3mm_M5_ISO7380, MountingHole:MountingHole_5.3mm_M5_ISO7380, F.Cu at (31.5, 180.2)
- added REF**: MountingHole_3.2mm_M3_ISO7380, MountingHole:MountingHole_3.2mm_M3_ISO7380, F.Cu at (77.5, 255.8)
- added REF**: MountingHole_3.2mm_M3_ISO7380, MountingHole:MountingHole_3.2mm_M3_ISO7380, F.Cu at (98.2, 235.5)
- added REF**: MountingHole_5.3mm_M5_ISO7380, MountingHole:MountingHole_5.3mm_M5_ISO7380, F.Cu at (46.8, 238.8)
- added REF**: MountingHole_3.2mm_M3_ISO7380, MountingHole:MountingHole_3.2mm_M3_ISO7380, F.Cu at (78.5, 209.5)
- added REF**: MountingHole_3.2mm_M3_ISO7380, MountingHole:MountingHole_3.2mm_M3_ISO7380, B.Cu at (280.8, 189.8)
- added REF**: MountingHole_3.2mm_M3_ISO7380, MountingHole:MountingHole_3.2mm_M3_ISO7380, F.Cu at (140.0, 256.2)
- added REF**: MountingHole_3.2mm_M3_ISO7380, MountingHole:MountingHole_3.2mm_M3_ISO7380, F.Cu at (98.2, 197.5)
- added REF**: MountingHole_5.3mm_M5_ISO7380, MountingHole:MountingHole_5.3mm_M5_ISO7380, F.Cu at (130.0, 238.8)
- added REF**: MountingHole_3.2mm_M3_ISO7380, MountingHole:MountingHole_3.2mm_M3_ISO7380, F.Cu at (40.2, 162.8)
- added REF**: MountingHole_3.2mm_M3_ISO7380, MountingHole:MountingHole_3.2mm_M3_ISO7380, F.Cu at (78.5, 171.5)
- added REF**: MountingHole_3.2mm_M3_ISO7380, MountingHole:MountingHole_3.2mm_M3_ISO7380, F.Cu at (40.5, 223.5)
- added REF**: MountingHole_3.2mm_M3_ISO7380, MountingHole:MountingHole_3.2mm_M3_ISO7380, F.Cu at (42.0, 192.5)
- added REF**: MountingHole_3.2mm_M3_ISO7380, MountingHole:MountingHole_3.2mm_M3_ISO7380, B.Cu at (319.0, 181.0)
- added REF**: MountingHole_3.2mm_M3_ISO7380, MountingHole:MountingHole_3.2mm_M3_ISO7380, B.Cu at (280.8, 227.8)
- added REF**: MountingHole_5.3mm_M5_ISO7380, MountingHole:MountingHole_5.3mm_M5_ISO7380, B.Cu at (312.5, 257.0)
- added REF**: MountingHole_3.2mm_M3_ISO7380, MountingHole:MountingHole_3.2mm_M3_ISO7380, B.Cu at (281.8, 274.0)
- added REF**: MountingHole_3.2mm_M3_ISO7380, MountingHole:MountingHole_3.2mm_M3_ISO7380, B.Cu at (261.0, 215.8)
- added REF**: MountingHole_5.3mm_M5_ISO7380, MountingHole:MountingHole_5.3mm_M5_ISO7380, B.Cu at (254.5, 191.5)
- added REF**: MountingHole_5.3mm_M5_ISO7380, MountingHole:MountingHole_5.3mm_M5_ISO7380, B.Cu at (327.8, 198.5)
Routing:
- net (no net): track 0.00 -> 7125.2 mm, vias 0 -> 132
Other:
- board size 134.1 x 130.9 mm -> 318.2 x 282.6 mm

Commit message: Update
Parts:
- moved REF** 153.4 mm to (252.0, 105.2)
- moved REF** 153.4 mm to (341.5, 90.0)
- moved REF** 153.4 mm to (242.0, 122.8)
- moved REF** 153.4 mm to (340.0, 59.0)
- moved REF** 153.4 mm to (283.8, 102.0)
- moved REF** 153.4 mm to (303.5, 38.0)
- moved REF** 153.4 mm to (341.8, 29.2)
- moved REF** 153.4 mm to (303.5, 76.0)
- moved REF** 153.4 mm to (335.2, 105.2)
- moved REF** 153.4 mm to (304.5, 122.2)
- moved REF** 153.4 mm to (283.8, 64.0)
- moved REF** 153.4 mm to (277.2, 39.8)
- moved REF** 153.4 mm to (350.5, 46.8)
- moved REF** 29.0 mm to (104.8, 202.2)
- moved REF** 29.0 mm to (31.5, 209.2)
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Routing:
- net (no net): track 7125.2 -> 0.00 mm, vias 132 -> 0
Other:
- board size 318.2 x 282.6 mm -> 341 x 293.4 mm

Commit message: Mounting holes in schematic.
Parts:
- renumbered REF** to H1, REF** to H10, REF** to H11, REF** to H12, REF** to H13, REF** to H14, REF** to H15, REF** to H16, REF** to H17, REF** to H18, REF** to H19, REF** to H2, REF** to H20, REF** to H21, REF** to H22, REF** to H23, REF** to H24, REF** to H25, REF** to H26, REF** to H3, REF** to H4, REF** to H5, REF** to H6, REF** to H7, REF** to H8, REF** to H9
Routing:
- net +5V: track 785.2 -> 926.4 mm
- net GND: track 662.5 -> 728.5 mm

Commit message: Update
Parts:
- H1, H14, H15, H16, H17, H2, H3, H4: value MountingHole_5.3mm_M5_ISO7380 -> MountingHole
- H10, H11, H12, H13, H18, H19, H20, H21, H22, H23, H24, H25, H26, H5, H6, H7, H8, H9: value MountingHole_3.2mm_M3_ISO7380 -> MountingHole
- moved H14 0.25 mm to (277.0, 39.8)
- moved H2 0.25 mm to (101.5, 39.8)

Commit message: Pcb progress
Routing:
- net +5V: track 926.4 -> 1560.0 mm
- net GND: track 728.5 -> 1293.3 mm

Commit message: Pcb progress
Parts:
- moved C19 3.95 mm to (126.5, 114.3)
- moved C1 3.95 mm to (27.0, 52.2)
- moved C10 3.95 mm to (64.5, 19.2)
- moved C11 3.95 mm to (64.5, 38.8)
- moved C12 3.95 mm to (64.5, 57.2)
- moved C13 3.95 mm to (64.5, 76.8)
- moved C14 3.95 mm to (102.5, 102.3)
- moved C15 3.95 mm to (83.0, 26.2)
- moved C16 3.95 mm to (83.0, 45.8)
- moved C17 3.95 mm to (83.0, 64.2)
- moved C18 3.95 mm to (83.5, 83.2)
- moved C2 3.95 mm to (27.0, 71.2)
- moved C20 3.95 mm to (103.0, 45.2)
- moved C21 3.95 mm to (102.5, 64.8)
- moved C22 3.95 mm to (102.0, 83.2)
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Routing:
- net +5V: track 1560.0 -> 1413.5 mm
- net /rcol3: track 0.00 -> 113.6 mm
- net /rcol1: track 0.00 -> 111.0 mm
- net /rcol2: track 0.00 -> 108.8 mm
- net /rcol0: track 0.00 -> 94.2 mm
- net /rrow1: track 0.00 -> 92.9 mm, vias 0 -> 8
- net /rrow2: track 0.00 -> 91.2 mm, vias 0 -> 7
- net /rrow3: track 0.00 -> 88.8 mm, vias 0 -> 3
- net /rcol4: track 0.00 -> 84.2 mm
- net /rrow4: track 0.00 -> 78.4 mm
- net /rrow0: track 0.00 -> 71.0 mm
- net GND: track 1293.3 -> 1223.3 mm
- net Net-(LED24-Pad4): track 0.00 -> 22.0 mm
- net Net-(LED28-Pad4): track 0.00 -> 9.37 mm
- net Net-(D42-Pad2): track 0.00 -> 4.40 mm
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Other:
- board size 341 x 293.4 mm -> 344.8 x 294.6 mm

Commit message: Pcb progress
Routing:
- net /rcol4: track 84.2 -> 182.8 mm, vias 0 -> 1
- net +5V: track 1413.5 -> 1496.7 mm
- net /rcol3: track 113.6 -> 195.9 mm, vias 0 -> 1
- net /rrow4: track 78.4 -> 157.1 mm
- net /rcol2: track 108.8 -> 184.8 mm, vias 0 -> 1
- net Net-(LED26-Pad4): track 0.00 -> 73.1 mm, vias 0 -> 2
- net /rrow0: track 71.0 -> 127.1 mm
- net /rcol1: track 111.0 -> 166.5 mm, vias 0 -> 1
- net /rrow3: track 88.8 -> 136.0 mm, vias 3 -> 5
- net /rcol0: track 94.2 -> 141.0 mm, vias 0 -> 1
- net Net-(LED38-Pad2): track 0.00 -> 40.6 mm, vias 0 -> 2
- net Net-(LED44-Pad2): track 0.00 -> 39.0 mm
- net /rrow2: track 91.2 -> 129.8 mm
- net /rrow1: track 92.9 -> 124.8 mm
- net /rSCL: track 0.00 -> 28.5 mm, vias 0 -> 1
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