File: pcb/memekbd.kicad_pcb (KiCad board)
At the start: 2 copper layers, 347.1 x 301.1 mm, 271 parts, among them J1 AudioJack4, J2 AudioJack4, SW1 SW_Push, SW10 SW_Push, SW11 SW_Push, SW12 SW_Push, SW13 SW_Push, SW14 SW_Push, SW15 SW_Push, SW16 SW_Push, SW17 SW_Push, SW18 SW_Push, SW19 SW_Push, SW2 KEY_SWITCH, SW2 SW_Push, SW20 SW_Push, SW21 SW_Push, SW22 SW_Push, SW23 SW_Push, SW24 SW_Push, SW25 SW_Push, SW26 SW_Push, SW27 SW_Push, SW28 SW_Push, SW29 SW_Push, SW3 SW_Push, SW30 SW_Push, SW31 SW_Push, SW32 SW_Push, SW33 SW_Push, SW34 SW_Push, SW35 SW_Push, SW36 SW_Push, SW37 SW_Push, SW38 SW_Push, SW39 SW_Push, SW4 SW_Push, SW40 SW_Push, SW41 SW_Push, SW42 SW_Push, SW43 SW_Push, SW44 SW_Push, SW45 SW_Push, SW46 SW_Push, SW47 SW_Push, SW48 SW_Push, SW5 SW_Push, SW6 SW_Push, SW7 SW_Push, SW8 SW_Push, SW9 SW_Push, U1 ProMicro, U2 ProMicro

Commit message: Fix refs
Parts:
- renumbered SW2 to REF**, H9 to REF**, H1 to REF**, H2 to REF**, H13 to REF**, H12 to REF**, H8 to REF**, H11 to REF**, H4 to REF**, H3 to REF**, H10 to REF**, H5 to REF**, H6 to REF**, H7 to REF**

Commit message: Update pcb
Connections:
- LED15 pad 2: Net-(LED15-Pad2) -> Net-(LED1-Pad4)
- LED20 pad 2: Net-(LED20-Pad2) -> Net-(LED2-Pad4)
- LED21 pad 2: Net-(LED20-Pad2) -> Net-(LED21-Pad2)
- LED23 pad 2: Net-(LED22-Pad2) -> Net-(LED23-Pad2)
- LED25 pad 4: Net-(LED24-Pad4) -> Net-(LED25-Pad4)
- LED27 pad 4: Net-(LED26-Pad4) -> Net-(LED27-Pad4)
- LED3 pad 4: Net-(LED2-Pad4) -> Net-(LED21-Pad2)
- LED38 pad 2: Net-(LED38-Pad2) -> Net-(LED24-Pad4)
- LED4 pad 4: Net-(LED4-Pad4) -> Net-(LED22-Pad2)
- LED43 pad 2: Net-(LED38-Pad2) -> Net-(LED25-Pad4)
- LED44 pad 2: Net-(LED44-Pad2) -> Net-(LED26-Pad4)
- LED45 pad 2: Net-(LED44-Pad2) -> Net-(LED27-Pad4)
- LED5 pad 4: Net-(LED1-Pad4) -> Net-(LED5-Pad4)
- R5 pad 1: Net-(LED15-Pad2) -> Net-(LED5-Pad4)

Commit message: Update pcb
Parts:
- moved R5 62.9 mm to (29.8, 32.2)
- moved R6 62.9 mm to (312.8, 34.5)
Routing:
- net Net-(LED26-Pad4): track 73.3 -> 0.00 mm, vias 2 -> 0
- net Net-(LED22-Pad2): track 70.6 -> 0.00 mm, vias 2 -> 0
- net Net-(LED1-Pad4): track 42.0 -> 0.00 mm, vias 2 -> 0
- net /lLED: track 40.9 -> 0.00 mm
- net Net-(LED38-Pad2): track 40.6 -> 0.00 mm, vias 2 -> 0
- net Net-(LED44-Pad2): track 39.0 -> 0.00 mm
- net Net-(LED20-Pad2): track 30.1 -> 0.00 mm, vias 2 -> 0
- net /rLED: track 25.5 -> 0.00 mm
- net Net-(LED2-Pad4): track 23.0 -> 0.00 mm, vias 2 -> 0
- net Net-(LED24-Pad4): track 22.7 -> 0.00 mm, vias 2 -> 0
- net Net-(LED28-Pad4): track 9.37 -> 0.00 mm
- net Net-(LED15-Pad2): track 8.79 -> 0.00 mm, vias 1 -> 0

Commit message: Re-finish manual layout
Parts:
- moved R6 62.9 mm to (250.0, 30.1)
Routing:
- net Net-(LED27-Pad4): track 0.00 -> 161.8 mm, vias 0 -> 2
- net Net-(LED2-Pad4): track 0.00 -> 116.7 mm, vias 0 -> 4
- net Net-(LED21-Pad2): track 0.00 -> 114.2 mm, vias 0 -> 4
- net /lLED: track 0.00 -> 109.6 mm, vias 0 -> 3
- net Net-(LED25-Pad4): track 0.00 -> 96.5 mm, vias 0 -> 2
- net Net-(LED26-Pad4): track 0.00 -> 94.2 mm, vias 0 -> 2
- net Net-(LED22-Pad2): track 0.00 -> 85.5 mm, vias 0 -> 2
- net Net-(LED1-Pad4): track 0.00 -> 84.7 mm, vias 0 -> 4
- net Net-(LED24-Pad4): track 0.00 -> 81.6 mm, vias 0 -> 2
- net Net-(LED5-Pad4): track 0.00 -> 13.8 mm, vias 0 -> 1
- net +5V: track 1689.4 -> 1682.7 mm
- net /rrow4: track 157.1 -> 151.2 mm, vias 2 -> 3
- net /lcol0: track 182.6 -> 186.4 mm
- net /rcol3: track 200.0 -> 202.9 mm, vias 5 -> 9
- net GND: track 1324.7 -> 1325.7 mm
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
Commit message: Update
Other:
- net class Default removed
- net class Power removed

Commit message: Update
Other:
- rule pad_to_mask_clearance: 0.05 -> 0
Changed lines of the file:
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@@
-(kicad_pcb (version 20210623) (generator pcbnew)
+(kicad_pcb (version 20210722) (generator pcbnew)
   (general
     (thickness 1.6)
@@
   )
   (setup
-    (pad_to_mask_clearance 0.05)
+    (stackup
+      (layer "F.SilkS" (type "Top Silk Screen"))
+      (layer "F.Paste" (type "Top Solder Paste"))
+      (layer "F.Mask" (type "Top Solder Mask") (color "Green") (thickness 0.01))
+      (layer "F.Cu" (type "copper") (thickness 0.035))
+      (layer "dielectric 1" (type "core") (thickness 1.51) (material "FR4") (epsilon_r 4.5) (loss_tangent 0.02))
+      (layer "B.Cu" (type "copper") (thickness 0.035))
+      (layer "B.Mask" (type "Bottom Solder Mask") (color "Green") (thickness 0.01))
+      (layer "B.Paste" (type "Bottom Solder Paste"))
+      (layer "B.SilkS" (type "Bottom Silk Screen"))
+      (copper_finish "None")
+      (dielectric_constraints no)
+    )
+    (pad_to_mask_clearance 0)
     (pcbplotparams
       (layerselection 0x00010fc_ffffffff)

Commit message: Update
Parts:
- added REF**: TestPoint_Pad_1.0x1.0mm, TestPoint:TestPoint_Pad_1.0x1.0mm, F.Cu at (143.8, 309.2)
- added REF**: TestPoint_Pad_1.0x1.0mm, TestPoint:TestPoint_Pad_1.0x1.0mm, F.Cu at (241.0, 206.5)
- added REF**: TestPoint_Pad_1.0x1.0mm, TestPoint:TestPoint_Pad_1.0x1.0mm, B.Cu at (143.8, 309.2)
- added REF**: TestPoint_Pad_1.0x1.0mm, TestPoint:TestPoint_Pad_1.0x1.0mm, B.Cu at (241.0, 206.5)
Changed lines of the file:
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@@
       (layerselection 0x00010fc_ffffffff)
       (disableapertmacros false)
-      (usegerberextensions false)
+      (usegerberextensions true)
       (usegerberattributes true)
       (usegerberadvancedattributes true)
@@
     (fp_line (start -9.525 -9.525) (end -9.525 9.525) (layer "F.Fab") (width 0.15))
   )
+  (footprint "TestPoint:TestPoint_Pad_1.0x1.0mm" (layer "F.Cu")
+    (at 143.75 309.25)
+    (descr "SMD rectangular pad as test Point, square 1.0mm side length")
+    (tags "test point SMD pad rectangle square")
+    (attr exclude_from_pos_files exclude_from_bom)
+    (fp_text reference "REF**" (at 0 -1.448) (layer "F.SilkS")
+      (effects (font (size 1 1) (thickness 0.15)))
+    )
+    (fp_text value "TestPoint_Pad_1.0x1.0mm" (at 0 1.55) (layer "F.Fab")
+      (effects (font (size 1 1) (thickness 0.15)))
+    )
+    (fp_text user "${REFERENCE}" (at 0 -1.45) (layer "F.Fab")
+      (effects (font (size 1 1) (thickness 0.15)))
+    )
+    (fp_line (start 0.7 -0.7) (end 0.7 0.7) (layer "F.SilkS") (width 0.12))
+    (fp_line (start 0.7 0.7) (end -0.7 0.7) (layer "F.SilkS") (width 0.12))
+    (fp_line (start -0.7 -0.7) (end 0.7 -0.7) (layer "F.SilkS") (width 0.12))
+    (fp_line (start -0.7 0.7) (end -0.7 -0.7) (layer "F.SilkS") (width 0.12))
+    (fp_line (start -1 -1) (end -1 1) (layer "F.CrtYd") (width 0.05))
+    (fp_line (start -1 -1) (end 1 -1) (layer "F.CrtYd") (width 0.05))
+    (fp_line (start 1 1) (end -1 1) (layer "F.CrtYd") (width 0.05))
+    (fp_line (start 1 1) (end 1 -1) (layer "F.CrtYd") (width 0.05))
+    (pad "1" smd rect locked (at 0 0) (size 1 1) (layers "F.Cu" "F.Mask"))
+  )
+  (footprint "TestPoint:TestPoint_Pad_1.0x1.0mm" (layer "F.Cu")
+    (at 241 206.5)
+    (descr "SMD rectangular pad as test Point, square 1.0mm side length")
+    (tags "test point SMD pad rectangle square")
+    (attr exclude_from_pos_files exclude_from_bom)
+    (fp_text reference "REF**" (at 0 -1.448) (layer "F.SilkS")
+      (effects (font (size 1 1) (thickness 0.15)))
+    )
+    (fp_text value "TestPoint_Pad_1.0x1.0mm" (at 0 1.55) (layer "F.Fab")
+      (effects (font (size 1 1) (thickness 0.15)))
+    )
+    (fp_text user "${REFERENCE}" (at 0 -1.45) (layer "F.Fab")
+      (effects (font (size 1 1) (thickness 0.15)))
+    )
+    (fp_line (start 0.7 -0.7) (end 0.7 0.7) (layer "F.SilkS") (width 0.12))
+    (fp_line (start -0.7 0.7) (end -0.7 -0.7) (layer "F.SilkS") (width 0.12))
+    (fp_line (start -0.7 -0.7) (end 0.7 -0.7) (layer "F.SilkS") (width 0.12))
+    (fp_line (start 0.7 0.7) (end -0.7 0.7) (layer "F.SilkS") (width 0.12))
+    (fp_line (start -1 -1) (end -1 1) (layer "F.CrtYd") (width 0.05))
+    (fp_line (start 1 1) (end -1 1) (layer "F.CrtYd") (width 0.05))
+    (fp_line (start 1 1) (end 1 -1) (layer "F.CrtYd") (width 0.05))
+    (fp_line (start -1 -1) (end 1 -1) (layer "F.CrtYd") (width 0.05))
+    (pad "1" smd rect locked (at 0 0) (size 1 1) (layers "F.Cu" "F.Mask"))
+  )
   (footprint "Capacitor_THT:C_Disc_D6.0mm_W2.5mm_P5.00mm" (layer "B.Cu")
     (at 244.5 47.5 180)
@@
     )
   )
+  (footprint "TestPoint:TestPoint_Pad_1.0x1.0mm" (layer "B.Cu")
+    (at 143.75 309.25 180)
+    (descr "SMD rectangular pad as test Point, square 1.0mm side length")
+    (tags "test point SMD pad rectangle square")
+    (attr exclude_from_pos_files exclude_from_bom)
+    (fp_text reference "REF**" (at 0 1.448) (layer "B.SilkS")
+      (effects (font (size 1 1) (thickness 0.15)) (justify mirror))
+    )
+    (fp_text value "TestPoint_Pad_1.0x1.0mm" (at 0 -1.55) (layer "B.Fab")
+      (effects (font (size 1 1) (thickness 0.15)) (justify mirror))
+    )
+    (fp_text user "${REFERENCE}" (at 0 1.45) (layer "B.Fab")
+      (effects (font (size 1 1) (thickness 0.15)) (justify mirror))
+    )
+    (fp_line (start -0.7 -0.7) (end -0.7 0.7) (layer "B.SilkS") (width 0.12))
+    (fp_line (start 0.7 0.7) (end 0.7 -0.7) (layer "B.SilkS") (width 0.12))
+    (fp_line (start -0.7 0.7) (end 0.7 0.7) (layer "B.SilkS") (width 0.12))
+    (fp_line (start 0.7 -0.7) (end -0.7 -0.7) (layer "B.SilkS") (width 0.12))
+    (fp_line (start -1 1) (end 1 1) (layer "B.CrtYd") (width 0.05))
+    (fp_line (start 1 -1) (end -1 -1) (layer "B.CrtYd") (width 0.05))
+    (fp_line (start -1 1) (end -1 -1) (layer "B.CrtYd") (width 0.05))
+    (fp_line (start 1 -1) (end 1 1) (layer "B.CrtYd") (width 0.05))
+    (pad "1" smd rect locked (at 0 0 180) (size 1 1) (layers "B.Cu" "B.Mask"))
+  )
+  (footprint "TestPoint:TestPoint_Pad_1.0x1.0mm" (layer "B.Cu")
+    (at 241 206.5 180)
+    (descr "SMD rectangular pad as test Point, square 1.0mm side length")
+    (tags "test point SMD pad rectangle square")
+    (attr exclude_from_pos_files exclude_from_bom)
+    (fp_text reference "REF**" (at 0 1.448) (layer "B.SilkS")
+      (effects (font (size 1 1) (thickness 0.15)) (justify mirror))
+    )
+    (fp_text value "TestPoint_Pad_1.0x1.0mm" (at 0 -1.55) (layer "B.Fab")
+      (effects (font (size 1 1) (thickness 0.15)) (justify mirror))
+    )
+    (fp_text user "${REFERENCE}" (at 0 1.45) (layer "B.Fab")
+      (effects (font (size 1 1) (thickness 0.15)) (justify mirror))
+    )
+    (fp_line (start -0.7 -0.7) (end -0.7 0.7) (layer "B.SilkS") (width 0.12))
+    (fp_line (start 0.7 0.7) (end 0.7 -0.7) (layer "B.SilkS") (width 0.12))
+    (fp_line (start 0.7 -0.7) (end -0.7 -0.7) (layer "B.SilkS") (width 0.12))
+    (fp_line (start -0.7 0.7) (end 0.7 0.7) (layer "B.SilkS") (width 0.12))
+    (fp_line (start -1 1) (end -1 -1) (layer "B.CrtYd") (width 0.05))
+    (fp_line (start 1 -1) (end 1 1) (layer "B.CrtYd") (width 0.05))
+    (fp_line (start -1 1) (end 1 1) (layer "B.CrtYd") (width 0.05))
+    (fp_line (start 1 -1) (end -1 -1) (layer "B.CrtYd") (width 0.05))
+    (pad "1" smd rect locked (at 0 0 180) (size 1 1) (layers "B.Cu" "B.Mask"))
+  )
   (gr_arc (start 79.5 181.5) (end 80 181.5) (angle -90) (layer "Edge.Cuts") (width 0.05))
