File: pcb/top_plate.kicad_pcb (KiCad board)
At the start: 2 copper layers, 134.1 x 130.9 mm, 36 parts, among them SW2 KEY_SWITCH

Commit message: Update subpcbs
Parts:
- added C1: 0.1uF, Capacitor_THT:C_Disc_D6.0mm_W2.5mm_P5.00mm, B.Cu at (27.0, 52.2)
- added C10: 0.1uF, Capacitor_THT:C_Disc_D6.0mm_W2.5mm_P5.00mm, B.Cu at (64.5, 19.2)
- added C11: 0.1uF, Capacitor_THT:C_Disc_D6.0mm_W2.5mm_P5.00mm, B.Cu at (64.5, 38.8)
- added C12: 0.1uF, Capacitor_THT:C_Disc_D6.0mm_W2.5mm_P5.00mm, B.Cu at (64.5, 57.2)
- added C13: 0.1uF, Capacitor_THT:C_Disc_D6.0mm_W2.5mm_P5.00mm, B.Cu at (64.5, 76.8)
- added C14: 0.1uF, Capacitor_THT:C_Disc_D6.0mm_W2.5mm_P5.00mm, B.Cu at (102.5, 102.3)
- added C15: 0.1uF, Capacitor_THT:C_Disc_D6.0mm_W2.5mm_P5.00mm, B.Cu at (83.0, 26.2)
- added C16: 0.1uF, Capacitor_THT:C_Disc_D6.0mm_W2.5mm_P5.00mm, B.Cu at (83.0, 45.8)
- added C17: 0.1uF, Capacitor_THT:C_Disc_D6.0mm_W2.5mm_P5.00mm, B.Cu at (83.0, 64.2)
- added C18: 0.1uF, Capacitor_THT:C_Disc_D6.0mm_W2.5mm_P5.00mm, B.Cu at (83.5, 83.2)
- added C19: 0.1uF, Capacitor_THT:C_Disc_D6.0mm_W2.5mm_P5.00mm, B.Cu at (126.5, 114.3)
- added C2: 0.1uF, Capacitor_THT:C_Disc_D6.0mm_W2.5mm_P5.00mm, B.Cu at (27.0, 71.2)
- added C20: 0.1uF, Capacitor_THT:C_Disc_D6.0mm_W2.5mm_P5.00mm, B.Cu at (103.0, 45.2)
- added C21: 0.1uF, Capacitor_THT:C_Disc_D6.0mm_W2.5mm_P5.00mm, B.Cu at (102.5, 64.8)
- added C22: 0.1uF, Capacitor_THT:C_Disc_D6.0mm_W2.5mm_P5.00mm, B.Cu at (102.0, 83.2)
- added C23: 0.1uF, Capacitor_THT:C_Disc_D6.0mm_W2.5mm_P5.00mm, B.Cu at (142.9, 131.0)
- added C24: 0.1uF, Capacitor_THT:C_Disc_D6.0mm_W2.5mm_P5.00mm, B.Cu at (244.5, 47.5)
- added C25: 0.1uF, Capacitor_THT:C_Disc_D6.0mm_W2.5mm_P5.00mm, B.Cu at (244.5, 66.5)
- added C26: 0.1uF, Capacitor_THT:C_Disc_D6.0mm_W2.5mm_P5.00mm, B.Cu at (244.0, 85.5)
- added C27: 0.1uF, Capacitor_THT:C_Disc_D6.0mm_W2.5mm_P5.00mm, B.Cu at (202.5, 130.4)
- added C28: 0.1uF, Capacitor_THT:C_Disc_D6.0mm_W2.5mm_P5.00mm, B.Cu at (263.5, 28.4)
- added C29: 0.1uF, Capacitor_THT:C_Disc_D6.0mm_W2.5mm_P5.00mm, B.Cu at (263.0, 47.5)
- added C3: 0.1uF, Capacitor_THT:C_Disc_D6.0mm_W2.5mm_P5.00mm, B.Cu at (27.0, 90.2)
- added C30: 0.1uF, Capacitor_THT:C_Disc_D6.0mm_W2.5mm_P5.00mm, B.Cu at (263.0, 67.0)
- added C31: 0.1uF, Capacitor_THT:C_Disc_D6.0mm_W2.5mm_P5.00mm, B.Cu at (263.0, 85.5)
- added C32: 0.1uF, Capacitor_THT:C_Disc_D6.0mm_W2.5mm_P5.00mm, B.Cu at (219.5, 114.6)
- added C33: 0.1uF, Capacitor_THT:C_Disc_D6.0mm_W2.5mm_P5.00mm, B.Cu at (282.0, 21.5)
- added C34: 0.1uF, Capacitor_THT:C_Disc_D6.0mm_W2.5mm_P5.00mm, B.Cu at (282.0, 40.5)
- added C35: 0.1uF, Capacitor_THT:C_Disc_D6.0mm_W2.5mm_P5.00mm, B.Cu at (281.5, 60.0)
- added C36: 0.1uF, Capacitor_THT:C_Disc_D6.0mm_W2.5mm_P5.00mm, B.Cu at (281.5, 78.5)
- added C37: 0.1uF, Capacitor_THT:C_Disc_D6.0mm_W2.5mm_P5.00mm, B.Cu at (243.5, 104.5)
- added C38: 0.1uF, Capacitor_THT:C_Disc_D6.0mm_W2.5mm_P5.00mm, B.Cu at (301.5, 23.5)
- added C39: 0.1uF, Capacitor_THT:C_Disc_D6.0mm_W2.5mm_P5.00mm, B.Cu at (301.0, 43.0)
- added C4: 0.1uF, Capacitor_THT:C_Disc_D6.0mm_W2.5mm_P5.00mm, B.Cu at (56.2, 107.3)
- added C40: 0.1uF, Capacitor_THT:C_Disc_D6.0mm_W2.5mm_P5.00mm, B.Cu at (301.0, 61.5)
- added C41: 0.1uF, Capacitor_THT:C_Disc_D6.0mm_W2.5mm_P5.00mm, B.Cu at (301.0, 80.5)
- added C42: 0.1uF, Capacitor_THT:C_Disc_D6.0mm_W2.5mm_P5.00mm, B.Cu at (267.7, 108.2)
- added C43: 0.1uF, Capacitor_THT:C_Disc_D6.0mm_W2.5mm_P5.00mm, B.Cu at (319.5, 55.0)
- added C44: 0.1uF, Capacitor_THT:C_Disc_D6.0mm_W2.5mm_P5.00mm, B.Cu at (320.5, 73.5)
- added C45: 0.1uF, Capacitor_THT:C_Disc_D6.0mm_W2.5mm_P5.00mm, B.Cu at (320.0, 92.5)
- added C46: 0.1uF, Capacitor_THT:C_Disc_D6.0mm_W2.5mm_P5.00mm, B.Cu at (290.2, 111.8)
- added C5: 0.1uF, Capacitor_THT:C_Disc_D6.0mm_W2.5mm_P5.00mm, B.Cu at (46.0, 21.2)
- added C6: 0.1uF, Capacitor_THT:C_Disc_D6.0mm_W2.5mm_P5.00mm, B.Cu at (46.0, 40.2)
- added C7: 0.1uF, Capacitor_THT:C_Disc_D6.0mm_W2.5mm_P5.00mm, B.Cu at (45.5, 59.8)
- added C8: 0.1uF, Capacitor_THT:C_Disc_D6.0mm_W2.5mm_P5.00mm, B.Cu at (45.5, 78.8)
- added C9: 0.1uF, Capacitor_THT:C_Disc_D6.0mm_W2.5mm_P5.00mm, B.Cu at (78.6, 104.9)
- added D1: 1N4148, Diode_THT:D_DO-35_SOD27_P7.62mm_Horizontal, B.Cu at (28.5, 68.8)
- added D10: 1N4148, Diode_THT:D_DO-35_SOD27_P7.62mm_Horizontal, B.Cu at (66.5, 35.8)
- added D11: 1N4148, Diode_THT:D_DO-35_SOD27_P7.62mm_Horizontal, B.Cu at (66.5, 54.8)
- added D12: 1N4148, Diode_THT:D_DO-35_SOD27_P7.62mm_Horizontal, B.Cu at (66.5, 73.8)
- added D13: 1N4148, Diode_THT:D_DO-35_SOD27_P7.62mm_Horizontal, B.Cu at (66.5, 92.8)
- added D14: 1N4148, Diode_THT:D_DO-35_SOD27_P7.62mm_Horizontal, B.Cu at (104.5, 118.8)
- added D15: 1N4148, Diode_THT:D_DO-35_SOD27_P7.62mm_Horizontal, B.Cu at (85.5, 42.8)
- added D16: 1N4148, Diode_THT:D_DO-35_SOD27_P7.62mm_Horizontal, B.Cu at (85.5, 61.8)
- added D17: 1N4148, Diode_THT:D_DO-35_SOD27_P7.62mm_Horizontal, B.Cu at (85.5, 80.8)
- added D18: 1N4148, Diode_THT:D_DO-35_SOD27_P7.62mm_Horizontal, B.Cu at (85.5, 99.8)
- added D19: 1N4148, Diode_THT:D_DO-35_SOD27_P7.62mm_Horizontal, B.Cu at (120.0, 129.6)
- added D2: 1N4148, Diode_THT:D_DO-35_SOD27_P7.62mm_Horizontal, B.Cu at (28.5, 87.8)
- added D20: 1N4148, Diode_THT:D_DO-35_SOD27_P7.62mm_Horizontal, B.Cu at (104.5, 61.8)
- added D21: 1N4148, Diode_THT:D_DO-35_SOD27_P7.62mm_Horizontal, B.Cu at (104.5, 80.8)
- added D22: 1N4148, Diode_THT:D_DO-35_SOD27_P7.62mm_Horizontal, B.Cu at (104.5, 99.8)
- added D23: 1N4148, Diode_THT:D_DO-35_SOD27_P7.62mm_Horizontal, B.Cu at (132.6, 144.1)
- added D24: 1N4148, Diode_THT:D_DO-35_SOD27_P7.62mm_Horizontal, B.Cu at (246.0, 64.0)
- added D25: 1N4148, Diode_THT:D_DO-35_SOD27_P7.62mm_Horizontal, B.Cu at (246.0, 83.0)
- added D26: 1N4148, Diode_THT:D_DO-35_SOD27_P7.62mm_Horizontal, B.Cu at (246.0, 102.0)
- added D27: 1N4148, Diode_THT:D_DO-35_SOD27_P7.62mm_Horizontal, B.Cu at (215.6, 140.7)
- added D28: 1N4148, Diode_THT:D_DO-35_SOD27_P7.62mm_Horizontal, B.Cu at (265.0, 45.0)
- added D29: 1N4148, Diode_THT:D_DO-35_SOD27_P7.62mm_Horizontal, B.Cu at (265.0, 64.0)
- added D3: 1N4148, Diode_THT:D_DO-35_SOD27_P7.62mm_Horizontal, B.Cu at (28.5, 106.8)
- added D30: 1N4148, Diode_THT:D_DO-35_SOD27_P7.62mm_Horizontal, B.Cu at (265.0, 83.0)
- added D31: 1N4148, Diode_THT:D_DO-35_SOD27_P7.62mm_Horizontal, B.Cu at (265.0, 102.0)
- added D32: 1N4148, Diode_THT:D_DO-35_SOD27_P7.62mm_Horizontal, B.Cu at (229.5, 127.9)
- added D33: 1N4148, Diode_THT:D_DO-35_SOD27_P7.62mm_Horizontal, B.Cu at (284.0, 38.0)
- added D34: 1N4148, Diode_THT:D_DO-35_SOD27_P7.62mm_Horizontal, B.Cu at (284.0, 57.0)
- added D35: 1N4148, Diode_THT:D_DO-35_SOD27_P7.62mm_Horizontal, B.Cu at (284.0, 76.0)
- added D36: 1N4148, Diode_THT:D_DO-35_SOD27_P7.62mm_Horizontal, B.Cu at (284.0, 95.0)
- added D37: 1N4148, Diode_THT:D_DO-35_SOD27_P7.62mm_Horizontal, B.Cu at (246.0, 121.0)
- added D38: 1N4148, Diode_THT:D_DO-35_SOD27_P7.62mm_Horizontal, B.Cu at (303.0, 40.0)
- added D39: 1N4148, Diode_THT:D_DO-35_SOD27_P7.62mm_Horizontal, B.Cu at (303.0, 59.0)
- added D4: 1N4148, Diode_THT:D_DO-35_SOD27_P7.62mm_Horizontal, B.Cu at (65.7, 120.9)
- added D40: 1N4148, Diode_THT:D_DO-35_SOD27_P7.62mm_Horizontal, B.Cu at (303.0, 78.0)
- added D41: 1N4148, Diode_THT:D_DO-35_SOD27_P7.62mm_Horizontal, B.Cu at (303.0, 97.0)
- added D42: 1N4148, Diode_THT:D_DO-35_SOD27_P7.62mm_Horizontal, B.Cu at (264.9, 124.5)
- added D43: 1N4148, Diode_THT:D_DO-35_SOD27_P7.62mm_Horizontal, B.Cu at (322.0, 71.0)
- added D44: 1N4148, Diode_THT:D_DO-35_SOD27_P7.62mm_Horizontal, B.Cu at (322.0, 90.0)
- added D45: 1N4148, Diode_THT:D_DO-35_SOD27_P7.62mm_Horizontal, B.Cu at (322.0, 109.0)
- added D46: 1N4148, Diode_THT:D_DO-35_SOD27_P7.62mm_Horizontal, B.Cu at (283.7, 127.1)
- added D5: 1N4148, Diode_THT:D_DO-35_SOD27_P7.62mm_Horizontal, B.Cu at (47.5, 37.8)
- added D6: 1N4148, Diode_THT:D_DO-35_SOD27_P7.62mm_Horizontal, B.Cu at (47.5, 56.8)
- added D7: 1N4148, Diode_THT:D_DO-35_SOD27_P7.62mm_Horizontal, B.Cu at (47.5, 75.8)
- added D8: 1N4148, Diode_THT:D_DO-35_SOD27_P7.62mm_Horizontal, B.Cu at (47.5, 94.8)
- added D9: 1N4148, Diode_THT:D_DO-35_SOD27_P7.62mm_Horizontal, B.Cu at (85.3, 120.2)
- added H1: MountingHole, MountingHole:MountingHole_5.3mm_M5_ISO7380, F.Cu at (24.2, 45.5)
- added H10: MountingHole, MountingHole:MountingHole_3.2mm_M3_ISO7380, F.Cu at (71.2, 36.8)
- added H11: MountingHole, MountingHole:MountingHole_3.2mm_M3_ISO7380, F.Cu at (70.2, 121.0)
- added H12: MountingHole, MountingHole:MountingHole_3.2mm_M3_ISO7380, F.Cu at (91.0, 100.8)
- added H13: MountingHole, MountingHole:MountingHole_3.2mm_M3_ISO7380, F.Cu at (132.8, 121.5)
- added H14: MountingHole, MountingHole:MountingHole_5.3mm_M5_ISO7380, B.Cu at (244.8, 40.8)
- added H15: MountingHole, MountingHole:MountingHole_5.3mm_M5_ISO7380, B.Cu at (318.2, 47.8)
- added H16: MountingHole, MountingHole:MountingHole_5.3mm_M5_ISO7380, B.Cu at (303.0, 106.2)
- added H17: MountingHole, MountingHole:MountingHole_5.3mm_M5_ISO7380, B.Cu at (219.8, 106.2)
- added H18: MountingHole, MountingHole:MountingHole_3.2mm_M3_ISO7380, B.Cu at (309.5, 30.2)
- added H19: MountingHole, MountingHole:MountingHole_3.2mm_M3_ISO7380, B.Cu at (307.8, 60.0)
- added H2: MountingHole, MountingHole:MountingHole_5.3mm_M5_ISO7380, F.Cu at (97.8, 38.5)
- added H20: MountingHole, MountingHole:MountingHole_3.2mm_M3_ISO7380, B.Cu at (309.2, 91.0)
- added H21: MountingHole, MountingHole:MountingHole_3.2mm_M3_ISO7380, B.Cu at (271.2, 39.0)
- added H22: MountingHole, MountingHole:MountingHole_3.2mm_M3_ISO7380, B.Cu at (271.2, 77.0)
- added H23: MountingHole, MountingHole:MountingHole_3.2mm_M3_ISO7380, B.Cu at (251.5, 65.0)
- added H24: MountingHole, MountingHole:MountingHole_3.2mm_M3_ISO7380, B.Cu at (251.5, 103.0)
- added H25: MountingHole, MountingHole:MountingHole_3.2mm_M3_ISO7380, B.Cu at (272.2, 123.2)
- added H26: MountingHole, MountingHole:MountingHole_3.2mm_M3_ISO7380, B.Cu at (209.8, 123.8)
- added H3: MountingHole, MountingHole:MountingHole_5.3mm_M5_ISO7380, F.Cu at (39.5, 104.0)
- added H4: MountingHole, MountingHole:MountingHole_5.3mm_M5_ISO7380, F.Cu at (122.8, 104.0)
- added H5: MountingHole, MountingHole:MountingHole_3.2mm_M3_ISO7380, F.Cu at (34.8, 57.8)
- added H6: MountingHole, MountingHole:MountingHole_3.2mm_M3_ISO7380, F.Cu at (33.2, 88.8)
- added H7: MountingHole, MountingHole:MountingHole_3.2mm_M3_ISO7380, F.Cu at (71.2, 74.8)
- added H8: MountingHole, MountingHole:MountingHole_3.2mm_M3_ISO7380, F.Cu at (91.0, 62.8)
- added H9: MountingHole, MountingHole:MountingHole_3.2mm_M3_ISO7380, F.Cu at (33.0, 28.0)
- added J1: AudioJack4, Connector_Audio:Jack_3.5mm_PJ320D_Horizontal, F.Cu at (119.5, 82.0)
- added J2: AudioJack4, Connector_Audio:Jack_3.5mm_PJ320D_Horizontal, F.Cu at (223.0, 84.5)
- added LED1: YS-SK6812MINI-E, kbd:YS-SK6812MINI-E, B.Cu at (24.5, 55.8)
- added LED10: YS-SK6812MINI-E, kbd:YS-SK6812MINI-E, B.Cu at (62.5, 22.8)
- added LED11: YS-SK6812MINI-E, kbd:YS-SK6812MINI-E, B.Cu at (62.5, 41.8)
- added LED12: YS-SK6812MINI-E, kbd:YS-SK6812MINI-E, B.Cu at (62.5, 60.8)
- added LED13: YS-SK6812MINI-E, kbd:YS-SK6812MINI-E, B.Cu at (62.5, 79.8)
- added LED14: YS-SK6812MINI-E, kbd:YS-SK6812MINI-E, B.Cu at (100.5, 105.8)
- added LED15: YS-SK6812MINI-E, kbd:YS-SK6812MINI-E, B.Cu at (81.5, 29.8)
- added LED16: YS-SK6812MINI-E, kbd:YS-SK6812MINI-E, B.Cu at (81.5, 48.8)
- added LED17: YS-SK6812MINI-E, kbd:YS-SK6812MINI-E, B.Cu at (81.5, 67.8)
- added LED18: YS-SK6812MINI-E, kbd:YS-SK6812MINI-E, B.Cu at (81.5, 86.8)
- added LED19: YS-SK6812MINI-E, kbd:YS-SK6812MINI-E, B.Cu at (123.0, 116.4)
- added LED2: YS-SK6812MINI-E, kbd:YS-SK6812MINI-E, B.Cu at (24.5, 74.8)
- added LED20: YS-SK6812MINI-E, kbd:YS-SK6812MINI-E, B.Cu at (100.5, 48.8)
- added LED21: YS-SK6812MINI-E, kbd:YS-SK6812MINI-E, B.Cu at (100.5, 67.8)
- added LED22: YS-SK6812MINI-E, kbd:YS-SK6812MINI-E, B.Cu at (100.5, 86.8)
- added LED23: YS-SK6812MINI-E, kbd:YS-SK6812MINI-E, B.Cu at (139.0, 132.1)
- added LED24: YS-SK6812MINI-E, kbd:YS-SK6812MINI-E, B.Cu at (242.0, 51.0)
- added LED25: YS-SK6812MINI-E, kbd:YS-SK6812MINI-E, B.Cu at (242.0, 70.0)
- added LED26: YS-SK6812MINI-E, kbd:YS-SK6812MINI-E, B.Cu at (242.0, 89.0)
- added LED27: YS-SK6812MINI-E, kbd:YS-SK6812MINI-E, B.Cu at (203.6, 134.3)
- added LED28: YS-SK6812MINI-E, kbd:YS-SK6812MINI-E, B.Cu at (261.0, 32.0)
- added LED29: YS-SK6812MINI-E, kbd:YS-SK6812MINI-E, B.Cu at (261.0, 51.0)
- added LED3: YS-SK6812MINI-E, kbd:YS-SK6812MINI-E, B.Cu at (24.5, 93.8)
- added LED30: YS-SK6812MINI-E, kbd:YS-SK6812MINI-E, B.Cu at (261.0, 70.0)
- added LED31: YS-SK6812MINI-E, kbd:YS-SK6812MINI-E, B.Cu at (261.0, 89.0)
- added LED32: YS-SK6812MINI-E, kbd:YS-SK6812MINI-E, B.Cu at (219.5, 118.6)
- added LED33: YS-SK6812MINI-E, kbd:YS-SK6812MINI-E, B.Cu at (280.0, 25.0)
- added LED34: YS-SK6812MINI-E, kbd:YS-SK6812MINI-E, B.Cu at (280.0, 44.0)
- added LED35: YS-SK6812MINI-E, kbd:YS-SK6812MINI-E, B.Cu at (280.0, 63.0)
- added LED36: YS-SK6812MINI-E, kbd:YS-SK6812MINI-E, B.Cu at (280.0, 82.0)
- added LED37: YS-SK6812MINI-E, kbd:YS-SK6812MINI-E, B.Cu at (242.0, 108.0)
- added LED38: YS-SK6812MINI-E, kbd:YS-SK6812MINI-E, B.Cu at (299.0, 27.0)
- added LED39: YS-SK6812MINI-E, kbd:YS-SK6812MINI-E, B.Cu at (299.0, 46.0)
- added LED4: YS-SK6812MINI-E, kbd:YS-SK6812MINI-E, B.Cu at (55.8, 111.6)
- added LED40: YS-SK6812MINI-E, kbd:YS-SK6812MINI-E, B.Cu at (299.0, 65.0)
- added LED41: YS-SK6812MINI-E, kbd:YS-SK6812MINI-E, B.Cu at (299.0, 84.0)
- added LED42: YS-SK6812MINI-E, kbd:YS-SK6812MINI-E, B.Cu at (264.4, 110.9)
- added LED43: YS-SK6812MINI-E, kbd:YS-SK6812MINI-E, B.Cu at (318.0, 58.0)
- added LED44: YS-SK6812MINI-E, kbd:YS-SK6812MINI-E, B.Cu at (318.0, 77.0)
- added LED45: YS-SK6812MINI-E, kbd:YS-SK6812MINI-E, B.Cu at (318.0, 96.0)
- added LED46: YS-SK6812MINI-E, kbd:YS-SK6812MINI-E, B.Cu at (286.8, 113.9)
- added LED5: YS-SK6812MINI-E, kbd:YS-SK6812MINI-E, B.Cu at (43.5, 24.8)
- added LED6: YS-SK6812MINI-E, kbd:YS-SK6812MINI-E, B.Cu at (43.5, 43.8)
- added LED7: YS-SK6812MINI-E, kbd:YS-SK6812MINI-E, B.Cu at (43.5, 62.8)
- added LED8: YS-SK6812MINI-E, kbd:YS-SK6812MINI-E, B.Cu at (43.5, 81.8)
- added LED9: YS-SK6812MINI-E, kbd:YS-SK6812MINI-E, B.Cu at (78.1, 108.7)
- added R1: 10k, Resistor_THT:R_Axial_DIN0207_L6.3mm_D2.5mm_P7.62mm_Horizontal, F.Cu at (119.5, 92.5)
- added R2: 10k, Resistor_THT:R_Axial_DIN0207_L6.3mm_D2.5mm_P7.62mm_Horizontal, F.Cu at (119.5, 89.0)
- added R3: 10k, Resistor_THT:R_Axial_DIN0207_L6.3mm_D2.5mm_P7.62mm_Horizontal, F.Cu at (223.0, 95.0)
- added R4: 10k, Resistor_THT:R_Axial_DIN0207_L6.3mm_D2.5mm_P7.62mm_Horizontal, F.Cu at (223.0, 91.5)
- added R5: 1k, Resistor_THT:R_Axial_DIN0207_L6.3mm_D2.5mm_P7.62mm_Horizontal, F.Cu at (92.5, 27.8)
- added R6: 1k, Resistor_THT:R_Axial_DIN0207_L6.3mm_D2.5mm_P7.62mm_Horizontal, F.Cu at (250.0, 30.0)
- added REF**: MountingHole_3.2mm_M3_ISO7380, MountingHole:MountingHole_3.2mm_M3_ISO7380, F.Cu at (140.8, 284.8)
- added REF**: MountingHole_3.2mm_M3_ISO7380, MountingHole:MountingHole_3.2mm_M3_ISO7380, F.Cu at (99.0, 264.0)
- added REF**: MountingHole_3.2mm_M3_ISO7380, MountingHole:MountingHole_3.2mm_M3_ISO7380, F.Cu at (41.2, 252.0)
- added REF**: MountingHole_5.3mm_M5_ISO7380, MountingHole:MountingHole_5.3mm_M5_ISO7380, F.Cu at (32.2, 208.8)
- added REF**: MountingHole_3.2mm_M3_ISO7380, MountingHole:MountingHole_3.2mm_M3_ISO7380, F.Cu at (99.0, 226.0)
- added REF**: MountingHole_3.2mm_M3_ISO7380, MountingHole:MountingHole_3.2mm_M3_ISO7380, F.Cu at (79.2, 200.0)
- added REF**: MountingHole_5.3mm_M5_ISO7380, MountingHole:MountingHole_5.3mm_M5_ISO7380, F.Cu at (105.5, 201.8)
- added REF**: MountingHole_3.2mm_M3_ISO7380, MountingHole:MountingHole_3.2mm_M3_ISO7380, F.Cu at (42.8, 221.0)
- added REF**: MountingHole_3.2mm_M3_ISO7380, MountingHole:MountingHole_3.2mm_M3_ISO7380, F.Cu at (79.2, 238.0)
- added REF**: MountingHole_3.2mm_M3_ISO7380, MountingHole:MountingHole_3.2mm_M3_ISO7380, F.Cu at (78.2, 284.2)
- added REF**: MountingHole_5.3mm_M5_ISO7380, MountingHole:MountingHole_5.3mm_M5_ISO7380, F.Cu at (47.5, 267.2)
- added REF**: MountingHole_3.2mm_M3_ISO7380, MountingHole:MountingHole_3.2mm_M3_ISO7380, F.Cu at (41.0, 191.2)
- added REF**: MountingHole_5.3mm_M5_ISO7380, MountingHole:MountingHole_5.3mm_M5_ISO7380, F.Cu at (130.8, 267.2)
- added SW1: SW_Push, kbd:CherryMX_Hotswap, F.Cu at (24.5, 60.2)
- added SW10: SW_Push, kbd:CherryMX_Hotswap, F.Cu at (62.5, 27.2)
- added SW11: SW_Push, kbd:CherryMX_Hotswap, F.Cu at (62.5, 46.2)
- added SW12: SW_Push, kbd:CherryMX_Hotswap, F.Cu at (62.5, 65.2)
- added SW13: SW_Push, kbd:CherryMX_Hotswap, F.Cu at (62.5, 84.2)
- added SW14: SW_Push, kbd:CherryMX_Hotswap, F.Cu at (100.5, 110.2)
- added SW15: SW_Push, kbd:CherryMX_Hotswap, F.Cu at (81.5, 34.2)
- added SW16: SW_Push, kbd:CherryMX_Hotswap, F.Cu at (81.5, 53.2)
- added SW17: SW_Push, kbd:CherryMX_Hotswap, F.Cu at (81.5, 72.2)
- added SW18: SW_Push, kbd:CherryMX_Hotswap, F.Cu at (81.5, 91.2)
- added SW19: SW_Push, kbd:CherryMX_Hotswap, F.Cu at (120.8, 120.2)
- added SW2: SW_Push, kbd:CherryMX_Hotswap, F.Cu at (24.5, 79.2)
- added SW20: SW_Push, kbd:CherryMX_Hotswap, F.Cu at (100.5, 53.2)
- added SW21: SW_Push, kbd:CherryMX_Hotswap, F.Cu at (100.5, 72.2)
- added SW22: SW_Push, kbd:CherryMX_Hotswap, F.Cu at (100.5, 91.2)
- added SW23: SW_Push, kbd:CherryMX_Hotswap, F.Cu at (135.8, 135.2)
- added SW24: SW_Push, kbd:CherryMX_Hotswap, F.Cu at (242.0, 55.5)
- added SW25: SW_Push, kbd:CherryMX_Hotswap, F.Cu at (242.0, 74.5)
- added SW26: SW_Push, kbd:CherryMX_Hotswap, F.Cu at (242.0, 93.5)
- added SW27: SW_Push, kbd:CherryMX_Hotswap, F.Cu at (206.8, 137.5)
- added SW28: SW_Push, kbd:CherryMX_Hotswap, F.Cu at (261.0, 36.5)
- added SW29: SW_Push, kbd:CherryMX_Hotswap, F.Cu at (261.0, 55.5)
- added SW3: SW_Push, kbd:CherryMX_Hotswap, F.Cu at (24.5, 98.2)
- added SW30: SW_Push, kbd:CherryMX_Hotswap, F.Cu at (261.0, 74.5)
- added SW31: SW_Push, kbd:CherryMX_Hotswap, F.Cu at (261.0, 93.5)
- added SW32: SW_Push, kbd:CherryMX_Hotswap, F.Cu at (221.8, 122.5)
- added SW33: SW_Push, kbd:CherryMX_Hotswap, F.Cu at (280.0, 29.5)
- added SW34: SW_Push, kbd:CherryMX_Hotswap, F.Cu at (280.0, 48.5)
- added SW35: SW_Push, kbd:CherryMX_Hotswap, F.Cu at (280.0, 67.5)
- added SW36: SW_Push, kbd:CherryMX_Hotswap, F.Cu at (280.0, 86.5)
- added SW37: SW_Push, kbd:CherryMX_Hotswap, F.Cu at (242.0, 112.5)
- added SW38: SW_Push, kbd:CherryMX_Hotswap, F.Cu at (299.0, 31.5)
- added SW39: SW_Push, kbd:CherryMX_Hotswap, F.Cu at (299.0, 50.5)
- added SW4: SW_Push, kbd:CherryMX_Hotswap, F.Cu at (58.0, 115.5)
- added SW40: SW_Push, kbd:CherryMX_Hotswap, F.Cu at (299.0, 69.5)
- added SW41: SW_Push, kbd:CherryMX_Hotswap, F.Cu at (299.0, 88.5)
- added SW42: SW_Push, kbd:CherryMX_Hotswap, F.Cu at (263.3, 115.2)
- added SW43: SW_Push, kbd:CherryMX_Hotswap, F.Cu at (318.0, 62.5)
- added SW44: SW_Push, kbd:CherryMX_Hotswap, F.Cu at (318.0, 81.5)
- added SW45: SW_Push, kbd:CherryMX_Hotswap, F.Cu at (318.0, 100.5)
- added SW46: SW_Push, kbd:CherryMX_Hotswap, F.Cu at (284.5, 117.8)
- added SW47: SW_Push, Button_Switch_THT:SW_PUSH_6mm_H7.3mm, F.Cu at (112.0, 95.5)
- added SW48: SW_Push, Button_Switch_THT:SW_PUSH_6mm_H7.3mm, F.Cu at (226.0, 98.0)
- added SW5: SW_Push, kbd:CherryMX_Hotswap, F.Cu at (43.5, 29.2)
- added SW6: SW_Push, kbd:CherryMX_Hotswap, F.Cu at (43.5, 48.2)
- added SW7: SW_Push, kbd:CherryMX_Hotswap, F.Cu at (43.5, 67.2)
- added SW8: SW_Push, kbd:CherryMX_Hotswap, F.Cu at (43.5, 86.2)
- added SW9: SW_Push, kbd:CherryMX_Hotswap, F.Cu at (79.2, 113.0)
- added U1: ProMicro, kbd:ProMicro_v3.5, F.Cu at (119.2, 62.0)
- added U2: ProMicro, kbd:ProMicro_v3.5, F.Cu at (223.2, 64.2)
- moved REF** 274.6 mm to (275.5, 254.5)
- moved REF** 274.6 mm to (237.5, 268.5)
- moved REF** 274.6 mm to (256.5, 237.5)
- moved REF** 274.6 mm to (348.8, 305.5)
- moved REF** 274.6 mm to (294.5, 223.5)
- moved REF** 274.6 mm to (294.5, 242.5)
- moved REF** 274.6 mm to (313.5, 280.5)
- moved REF** 274.6 mm to (313.5, 223.5)
- moved REF** 274.6 mm to (313.5, 242.5)
- moved REF** 274.6 mm to (294.5, 204.5)
- moved REF** 274.6 mm to (256.5, 218.5)
- moved REF** 274.6 mm to (275.5, 197.5)
- moved REF** 274.6 mm to (271.0, 285.8)
- moved REF** 274.6 mm to (237.5, 230.5)
- moved REF** 274.6 mm to (313.5, 261.5)
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- renumbered SW2 to REF**, H9 to REF**, H1 to REF**, H2 to REF**, H13 to REF**, H12 to REF**, H8 to REF**, H11 to REF**, H4 to REF**, H3 to REF**, H10 to REF**, H5 to REF**, H6 to REF**, H7 to REF**
Routing:
- net +5V: track 0.00 -> 1689.4 mm
- net GND: track 0.00 -> 1324.7 mm, vias 0 -> 1
- net /rcol3: track 0.00 -> 200.0 mm, vias 0 -> 5
- net /lcol1: track 0.00 -> 193.7 mm, vias 0 -> 6
- net /rcol4: track 0.00 -> 186.6 mm, vias 0 -> 3
- net /lcol0: track 0.00 -> 182.6 mm, vias 0 -> 3
- net /rcol2: track 0.00 -> 181.4 mm, vias 0 -> 4
- net /rcol1: track 0.00 -> 169.2 mm, vias 0 -> 5
- net /lcol3: track 0.00 -> 167.5 mm, vias 0 -> 3
- net /lcol2: track 0.00 -> 166.8 mm, vias 0 -> 3
- net /rrow4: track 0.00 -> 157.1 mm, vias 0 -> 2
- net /rcol0: track 0.00 -> 142.2 mm, vias 0 -> 3
- net /lcol4: track 0.00 -> 138.4 mm, vias 0 -> 2
- net /rrow3: track 0.00 -> 136.0 mm, vias 0 -> 5
- net /lrow4: track 0.00 -> 134.9 mm, vias 0 -> 2
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Other:
- board size 134.1 x 130.9 mm -> 347.1 x 301.1 mm

Commit message: Update
Parts:
- removed C1, C10, C11, C12, C13, C14, C15, C16, C17, C18, C19, C2, C20, C21, C22, C23, C24, C25, C26, C27, C28, C29, C3, C30, C31, C32, C33, C34, C35, C36, C37, C38, C39, C4, C40, C41, C42, C43, C44, C45, C46, C5, C6, C7, C8, C9: 0.1uF, Capacitor_THT:C_Disc_D6.0mm_W2.5mm_P5.00mm
- removed D1, D10, D11, D12, D13, D14, D15, D16, D17, D18, D19, D2, D20, D21, D22, D23, D24, D25, D26, D27, D28, D29, D3, D30, D31, D32, D33, D34, D35, D36, D37, D38, D39, D4, D40, D41, D42, D43, D44, D45, D46, D5, D6, D7, D8, D9: 1N4148, Diode_THT:D_DO-35_SOD27_P7.62mm_Horizontal
- removed H1, H14, H15, H16, H17, H2, H3, H4: MountingHole, MountingHole:MountingHole_5.3mm_M5_ISO7380
- removed H10, H11, H12, H13, H18, H19, H20, H21, H22, H23, H24, H25, H26, H5, H6, H7, H8, H9: MountingHole, MountingHole:MountingHole_3.2mm_M3_ISO7380
- removed J1, J2: AudioJack4, Connector_Audio:Jack_3.5mm_PJ320D_Horizontal
- removed LED1, LED10, LED11, LED12, LED13, LED14, LED15, LED16, LED17, LED18, LED19, LED2, LED20, LED21, LED22, LED23, LED24, LED25, LED26, LED27, LED28, LED29, LED3, LED30, LED31, LED32, LED33, LED34, LED35, LED36, LED37, LED38, LED39, LED4, LED40, LED41, LED42, LED43, LED44, LED45, LED46, LED5, LED6, LED7, LED8, LED9: YS-SK6812MINI-E, kbd:YS-SK6812MINI-E
- removed R1, R2, R3, R4: 10k, Resistor_THT:R_Axial_DIN0207_L6.3mm_D2.5mm_P7.62mm_Horizontal
- removed R5, R6: 1k, Resistor_THT:R_Axial_DIN0207_L6.3mm_D2.5mm_P7.62mm_Horizontal
- removed the REF** at (140.8, 284.8)
- removed the REF** at (99.0, 264.0)
- removed the REF** at (41.2, 252.0)
- removed the REF** at (32.2, 208.8)
- removed the REF** at (99.0, 226.0)
- removed the REF** at (79.2, 200.0)
- removed the REF** at (105.5, 201.8)
- removed the REF** at (42.8, 221.0)
- removed the REF** at (79.2, 238.0)
- removed the REF** at (78.2, 284.2)
- removed the REF** at (47.5, 267.2)
- removed the REF** at (41.0, 191.2)
- removed the REF** at (130.8, 267.2)
- removed SW1, SW10, SW11, SW12, SW13, SW14, SW15, SW16, SW17, SW18, SW19, SW2, SW20, SW21, SW22, SW23, SW24, SW25, SW26, SW27, SW28, SW29, SW3, SW30, SW31, SW32, SW33, SW34, SW35, SW36, SW37, SW38, SW39, SW4, SW40, SW41, SW42, SW43, SW44, SW45, SW46, SW5, SW6, SW7, SW8, SW9: SW_Push, kbd:CherryMX_Hotswap
- removed SW47, SW48: SW_Push, Button_Switch_THT:SW_PUSH_6mm_H7.3mm
- removed U1, U2: ProMicro, kbd:ProMicro_v3.5
- moved REF** 289.8 mm to (61.0, 60.2)
- moved REF** 289.8 mm to (47.8, 101.0)
- moved REF** 289.8 mm to (14.2, 83.8)
- moved REF** 289.8 mm to (71.2, 38.8)
- moved REF** 289.8 mm to (60.0, 106.5)
- moved REF** 289.8 mm to (90.2, 57.8)
- moved REF** 289.8 mm to (90.2, 76.8)
- moved REF** 289.8 mm to (24.5, 43.2)
- moved REF** 289.8 mm to (80.8, 86.2)
- moved REF** 289.8 mm to (52.2, 69.8)
- moved REF** 289.8 mm to (33.2, 71.8)
- moved REF** 289.8 mm to (90.2, 95.8)
- moved REF** 289.8 mm to (71.2, 57.8)
- moved REF** 289.8 mm to (52.2, 12.8)
- moved REF** 289.8 mm to (122.5, 107.0)
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Routing:
- net +5V: track 1689.4 -> 0.00 mm
- net GND: track 1324.7 -> 0.00 mm, vias 1 -> 0
- net /rcol3: track 200.0 -> 0.00 mm, vias 5 -> 0
- net /lcol1: track 193.7 -> 0.00 mm, vias 6 -> 0
- net /rcol4: track 186.6 -> 0.00 mm, vias 3 -> 0
- net /lcol0: track 182.6 -> 0.00 mm, vias 3 -> 0
- net /rcol2: track 181.4 -> 0.00 mm, vias 4 -> 0
- net /rcol1: track 169.2 -> 0.00 mm, vias 5 -> 0
- net /lcol3: track 167.5 -> 0.00 mm, vias 3 -> 0
- net /lcol2: track 166.8 -> 0.00 mm, vias 3 -> 0
- net /rrow4: track 157.1 -> 0.00 mm, vias 2 -> 0
- net /rcol0: track 142.2 -> 0.00 mm, vias 3 -> 0
- net /lcol4: track 138.4 -> 0.00 mm, vias 2 -> 0
- net /rrow3: track 136.0 -> 0.00 mm, vias 5 -> 0
- net /lrow4: track 134.9 -> 0.00 mm, vias 2 -> 0
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Other:
- board size 347.1 x 301.1 mm -> 134.1 x 130.9 mm
- net class Default removed
- net class Power removed

Commit message: Update
Other:
- rule pad_to_mask_clearance: 0.05 -> 0
Changed lines of the file:
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@@
-(kicad_pcb (version 20210623) (generator pcbnew)
+(kicad_pcb (version 20210722) (generator pcbnew)
   (general
     (thickness 1.6)
@@
   )
   (setup
-    (pad_to_mask_clearance 0.05)
+    (stackup
+      (layer "F.SilkS" (type "Top Silk Screen"))
+      (layer "F.Paste" (type "Top Solder Paste"))
+      (layer "F.Mask" (type "Top Solder Mask") (color "Green") (thickness 0.01))
+      (layer "F.Cu" (type "copper") (thickness 0.035))
+      (layer "dielectric 1" (type "core") (thickness 1.51) (material "FR4") (epsilon_r 4.5) (loss_tangent 0.02))
+      (layer "B.Cu" (type "copper") (thickness 0.035))
+      (layer "B.Mask" (type "Bottom Solder Mask") (color "Green") (thickness 0.01))
+      (layer "B.Paste" (type "Bottom Solder Paste"))
+      (layer "B.SilkS" (type "Bottom Silk Screen"))
+      (copper_finish "None")
+      (dielectric_constraints no)
+    )
+    (pad_to_mask_clearance 0)
     (pcbplotparams
       (layerselection 0x00010fc_ffffffff)
@@
       (drillshape 0)
       (scaleselection 1)
-      (outputdirectory "gerbers")
+      (outputdirectory "gerbers/top")
     )
   )
