File: pcb/left.kicad_pcb (KiCad board)
At the start: 2 copper layers, 347.1 x 301.1 mm, 271 parts, among them J1 AudioJack4, J2 AudioJack4, SW1 SW_Push, SW10 SW_Push, SW11 SW_Push, SW12 SW_Push, SW13 SW_Push, SW14 SW_Push, SW15 SW_Push, SW16 SW_Push, SW17 SW_Push, SW18 SW_Push, SW19 SW_Push, SW2 KEY_SWITCH, SW2 SW_Push, SW20 SW_Push, SW21 SW_Push, SW22 SW_Push, SW23 SW_Push, SW24 SW_Push, SW25 SW_Push, SW26 SW_Push, SW27 SW_Push, SW28 SW_Push, SW29 SW_Push, SW3 SW_Push, SW30 SW_Push, SW31 SW_Push, SW32 SW_Push, SW33 SW_Push, SW34 SW_Push, SW35 SW_Push, SW36 SW_Push, SW37 SW_Push, SW38 SW_Push, SW39 SW_Push, SW4 SW_Push, SW40 SW_Push, SW41 SW_Push, SW42 SW_Push, SW43 SW_Push, SW44 SW_Push, SW45 SW_Push, SW46 SW_Push, SW47 SW_Push, SW48 SW_Push, SW5 SW_Push, SW6 SW_Push, SW7 SW_Push, SW8 SW_Push, SW9 SW_Push, U1 ProMicro, U2 ProMicro

Commit message: Add other subparts
Parts:
- removed C24, C25, C26, C27, C28, C29, C30, C31, C32, C33, C34, C35, C36, C37, C38, C39, C40, C41, C42, C43, C44, C45, C46: 0.1uF, Capacitor_THT:C_Disc_D6.0mm_W2.5mm_P5.00mm
- removed D24, D25, D26, D27, D28, D29, D30, D31, D32, D33, D34, D35, D36, D37, D38, D39, D40, D41, D42, D43, D44, D45, D46: 1N4148, Diode_THT:D_DO-35_SOD27_P7.62mm_Horizontal
- removed the H1 at (237.2, 215.8)
- removed the H10 at (284.2, 207.0)
- removed the H11 at (283.2, 291.2)
- removed the H12 at (304.0, 271.0)
- removed the H13 at (345.8, 291.8)
- removed H14, H15, H16, H17: MountingHole, MountingHole:MountingHole_5.3mm_M5_ISO7380
- removed H18, H19, H20, H21, H22, H23, H24, H25, H26: MountingHole, MountingHole:MountingHole_3.2mm_M3_ISO7380
- removed the H2 at (310.8, 208.8)
- removed the H3 at (252.5, 274.2)
- removed the H4 at (335.8, 274.2)
- removed the H5 at (247.8, 228.0)
- removed the H6 at (246.2, 259.0)
- removed the H7 at (284.2, 245.0)
- removed the H8 at (304.0, 233.0)
- removed the H9 at (246.0, 198.2)
- removed J2: AudioJack4, Connector_Audio:Jack_3.5mm_PJ320D_Horizontal
- removed LED24, LED25, LED26, LED27, LED28, LED29, LED30, LED31, LED32, LED33, LED34, LED35, LED36, LED37, LED38, LED39, LED40, LED41, LED42, LED43, LED44, LED45, LED46: YS-SK6812MINI-E, kbd:YS-SK6812MINI-E
- removed R3, R4: 10k, Resistor_THT:R_Axial_DIN0207_L6.3mm_D2.5mm_P7.62mm_Horizontal
- removed R6: 1k, Resistor_THT:R_Axial_DIN0207_L6.3mm_D2.5mm_P7.62mm_Horizontal
- removed REF** (x9): MountingHole_3.2mm_M3_ISO7380, MountingHole:MountingHole_3.2mm_M3_ISO7380
- removed REF** (x4): MountingHole_5.3mm_M5_ISO7380, MountingHole:MountingHole_5.3mm_M5_ISO7380
- removed the SW2 at (275.5, 254.5)
- removed the SW2 at (237.5, 268.5)
- removed the SW2 at (256.5, 237.5)
- removed the SW2 at (348.8, 305.5)
- removed the SW2 at (294.5, 223.5)
- removed the SW2 at (294.5, 242.5)
- removed the SW2 at (313.5, 280.5)
- removed the SW2 at (313.5, 223.5)
- removed the SW2 at (313.5, 242.5)
- removed the SW2 at (294.5, 204.5)
- removed the SW2 at (256.5, 218.5)
- removed the SW2 at (275.5, 197.5)
- removed the SW2 at (271.0, 285.8)
- removed the SW2 at (237.5, 230.5)
- removed the SW2 at (313.5, 261.5)
- removed the SW2 at (275.5, 235.5)
- removed the SW2 at (256.5, 199.5)
- removed the SW2 at (275.5, 216.5)
- removed the SW2 at (256.5, 256.5)
- removed the SW2 at (294.5, 261.5)
- removed the SW2 at (333.8, 290.5)
- removed the SW2 at (292.2, 283.2)
- removed the SW2 at (237.5, 249.5)
- removed SW24, SW25, SW26, SW27, SW28, SW29, SW30, SW31, SW32, SW33, SW34, SW35, SW36, SW37, SW38, SW39, SW40, SW41, SW42, SW43, SW44, SW45, SW46: SW_Push, kbd:CherryMX_Hotswap
- removed SW48: SW_Push, Button_Switch_THT:SW_PUSH_6mm_H7.3mm
- removed U2: ProMicro, kbd:ProMicro_v3.5
Routing:
- net +5V: track 1689.4 -> 785.2 mm
- net GND: track 1324.7 -> 662.5 mm
- net /rcol3: track 200.0 -> 0.00 mm, vias 5 -> 0
- net /rcol4: track 186.6 -> 0.00 mm, vias 3 -> 0
- net /rcol2: track 181.4 -> 0.00 mm, vias 4 -> 0
- net /rcol1: track 169.2 -> 0.00 mm, vias 5 -> 0
- net /rrow4: track 157.1 -> 0.00 mm, vias 2 -> 0
- net /rcol0: track 142.2 -> 0.00 mm, vias 3 -> 0
- net /rrow3: track 136.0 -> 0.00 mm, vias 5 -> 0
- net /rrow2: track 129.8 -> 0.00 mm, vias 7 -> 0
- net /rrow1: track 124.8 -> 0.00 mm, vias 8 -> 0
- net /rrow0: track 109.1 -> 0.00 mm, vias 2 -> 0
- net Net-(LED26-Pad4): track 73.3 -> 0.00 mm, vias 2 -> 0
- net /rRST: track 50.5 -> 0.00 mm, vias 2 -> 0
- net /rSCL: track 43.7 -> 0.00 mm, vias 2 -> 0
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Other:
- board size 347.1 x 301.1 mm -> 134.1 x 130.9 mm

Commit message: Update subpcbs
Connections:
- LED15 pad 2: Net-(LED15-Pad2) -> Net-(LED1-Pad4)
- LED20 pad 2: Net-(LED20-Pad2) -> Net-(LED2-Pad4)
- LED21 pad 2: Net-(LED20-Pad2) -> Net-(LED21-Pad2)
- LED23 pad 2: Net-(LED22-Pad2) -> Net-(LED23-Pad2)
- LED3 pad 4: Net-(LED2-Pad4) -> Net-(LED21-Pad2)
- LED4 pad 4: Net-(LED4-Pad4) -> Net-(LED22-Pad2)
- LED5 pad 4: Net-(LED1-Pad4) -> Net-(LED5-Pad4)
- R5 pad 1: Net-(LED15-Pad2) -> Net-(LED5-Pad4)
Routing:
- net +5V: track 785.2 -> 0.00 mm
- net GND: track 662.5 -> 0.00 mm, vias 1 -> 0
- net /lcol1: track 193.7 -> 0.00 mm, vias 6 -> 0
- net /lcol0: track 182.6 -> 0.00 mm, vias 3 -> 0
- net /lcol3: track 167.5 -> 0.00 mm, vias 3 -> 0
- net /lcol2: track 166.8 -> 0.00 mm, vias 3 -> 0
- net /lcol4: track 138.4 -> 0.00 mm, vias 2 -> 0
- net /lrow4: track 134.9 -> 0.00 mm, vias 2 -> 0
- net /lrow3: track 124.7 -> 0.00 mm, vias 1 -> 0
- net /lrow2: track 106.6 -> 0.00 mm
- net /lrow1: track 93.4 -> 0.00 mm
- net /lrow0: track 78.5 -> 0.00 mm
- net Net-(LED22-Pad2): track 70.6 -> 0.00 mm, vias 2 -> 0
- net /lRST: track 45.3 -> 0.00 mm
- net Net-(LED1-Pad4): track 42.0 -> 0.00 mm, vias 2 -> 0
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
Commit message: Update
Other:
- net class Default removed
- net class Power removed

Commit message: Update
Parts:
- moved R5 62.9 mm to (29.8, 32.2)
Routing:
- net +5V: track 0.00 -> 784.9 mm
- net GND: track 0.00 -> 662.5 mm, vias 0 -> 1
- net /lcol1: track 0.00 -> 193.7 mm, vias 0 -> 6
- net /lcol0: track 0.00 -> 186.4 mm, vias 0 -> 3
- net /lcol3: track 0.00 -> 167.5 mm, vias 0 -> 3
- net /lcol2: track 0.00 -> 166.2 mm, vias 0 -> 5
- net /lcol4: track 0.00 -> 138.4 mm, vias 0 -> 2
- net /lrow4: track 0.00 -> 134.9 mm, vias 0 -> 2
- net /lrow3: track 0.00 -> 124.7 mm, vias 0 -> 1
- net Net-(LED2-Pad4): track 0.00 -> 116.7 mm, vias 0 -> 4
- net Net-(LED21-Pad2): track 0.00 -> 114.2 mm, vias 0 -> 4
- net /lLED: track 0.00 -> 109.6 mm, vias 0 -> 3
- net /lrow2: track 0.00 -> 106.6 mm
- net /lrow1: track 0.00 -> 93.4 mm
- net Net-(LED22-Pad2): track 0.00 -> 85.5 mm, vias 0 -> 2
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Other:
- rule pad_to_mask_clearance: 0.05 -> 0
