File: pcb/right.kicad_pcb (KiCad board)
At the start: 2 copper layers, 134.1 x 130.9 mm, 111 parts, among them J2 AudioJack4, SW24 SW_Push, SW25 SW_Push, SW26 SW_Push, SW27 SW_Push, SW28 SW_Push, SW29 SW_Push, SW30 SW_Push, SW31 SW_Push, SW32 SW_Push, SW33 SW_Push, SW34 SW_Push, SW35 SW_Push, SW36 SW_Push, SW37 SW_Push, SW38 SW_Push, SW39 SW_Push, SW40 SW_Push, SW41 SW_Push, SW42 SW_Push, SW43 SW_Push, SW44 SW_Push, SW45 SW_Push, SW46 SW_Push, SW48 SW_Push, U2 ProMicro

Commit message: Update subpcbs
Parts:
- added C1: 0.1uF, Capacitor_THT:C_Disc_D6.0mm_W2.5mm_P5.00mm, B.Cu at (27.0, 52.2)
- added C10: 0.1uF, Capacitor_THT:C_Disc_D6.0mm_W2.5mm_P5.00mm, B.Cu at (64.5, 19.2)
- added C11: 0.1uF, Capacitor_THT:C_Disc_D6.0mm_W2.5mm_P5.00mm, B.Cu at (64.5, 38.8)
- added C12: 0.1uF, Capacitor_THT:C_Disc_D6.0mm_W2.5mm_P5.00mm, B.Cu at (64.5, 57.2)
- added C13: 0.1uF, Capacitor_THT:C_Disc_D6.0mm_W2.5mm_P5.00mm, B.Cu at (64.5, 76.8)
- added C14: 0.1uF, Capacitor_THT:C_Disc_D6.0mm_W2.5mm_P5.00mm, B.Cu at (102.5, 102.3)
- added C15: 0.1uF, Capacitor_THT:C_Disc_D6.0mm_W2.5mm_P5.00mm, B.Cu at (83.0, 26.2)
- added C16: 0.1uF, Capacitor_THT:C_Disc_D6.0mm_W2.5mm_P5.00mm, B.Cu at (83.0, 45.8)
- added C17: 0.1uF, Capacitor_THT:C_Disc_D6.0mm_W2.5mm_P5.00mm, B.Cu at (83.0, 64.2)
- added C18: 0.1uF, Capacitor_THT:C_Disc_D6.0mm_W2.5mm_P5.00mm, B.Cu at (83.5, 83.2)
- added C19: 0.1uF, Capacitor_THT:C_Disc_D6.0mm_W2.5mm_P5.00mm, B.Cu at (126.5, 114.3)
- added C2: 0.1uF, Capacitor_THT:C_Disc_D6.0mm_W2.5mm_P5.00mm, B.Cu at (27.0, 71.2)
- added C20: 0.1uF, Capacitor_THT:C_Disc_D6.0mm_W2.5mm_P5.00mm, B.Cu at (103.0, 45.2)
- added C21: 0.1uF, Capacitor_THT:C_Disc_D6.0mm_W2.5mm_P5.00mm, B.Cu at (102.5, 64.8)
- added C22: 0.1uF, Capacitor_THT:C_Disc_D6.0mm_W2.5mm_P5.00mm, B.Cu at (102.0, 83.2)
- added C23: 0.1uF, Capacitor_THT:C_Disc_D6.0mm_W2.5mm_P5.00mm, B.Cu at (142.9, 131.0)
- added C3: 0.1uF, Capacitor_THT:C_Disc_D6.0mm_W2.5mm_P5.00mm, B.Cu at (27.0, 90.2)
- added C4: 0.1uF, Capacitor_THT:C_Disc_D6.0mm_W2.5mm_P5.00mm, B.Cu at (56.2, 107.3)
- added C5: 0.1uF, Capacitor_THT:C_Disc_D6.0mm_W2.5mm_P5.00mm, B.Cu at (46.0, 21.2)
- added C6: 0.1uF, Capacitor_THT:C_Disc_D6.0mm_W2.5mm_P5.00mm, B.Cu at (46.0, 40.2)
- added C7: 0.1uF, Capacitor_THT:C_Disc_D6.0mm_W2.5mm_P5.00mm, B.Cu at (45.5, 59.8)
- added C8: 0.1uF, Capacitor_THT:C_Disc_D6.0mm_W2.5mm_P5.00mm, B.Cu at (45.5, 78.8)
- added C9: 0.1uF, Capacitor_THT:C_Disc_D6.0mm_W2.5mm_P5.00mm, B.Cu at (78.6, 104.9)
- added D1: 1N4148, Diode_THT:D_DO-35_SOD27_P7.62mm_Horizontal, B.Cu at (28.5, 68.8)
- added D10: 1N4148, Diode_THT:D_DO-35_SOD27_P7.62mm_Horizontal, B.Cu at (66.5, 35.8)
- added D11: 1N4148, Diode_THT:D_DO-35_SOD27_P7.62mm_Horizontal, B.Cu at (66.5, 54.8)
- added D12: 1N4148, Diode_THT:D_DO-35_SOD27_P7.62mm_Horizontal, B.Cu at (66.5, 73.8)
- added D13: 1N4148, Diode_THT:D_DO-35_SOD27_P7.62mm_Horizontal, B.Cu at (66.5, 92.8)
- added D14: 1N4148, Diode_THT:D_DO-35_SOD27_P7.62mm_Horizontal, B.Cu at (104.5, 118.8)
- added D15: 1N4148, Diode_THT:D_DO-35_SOD27_P7.62mm_Horizontal, B.Cu at (85.5, 42.8)
- added D16: 1N4148, Diode_THT:D_DO-35_SOD27_P7.62mm_Horizontal, B.Cu at (85.5, 61.8)
- added D17: 1N4148, Diode_THT:D_DO-35_SOD27_P7.62mm_Horizontal, B.Cu at (85.5, 80.8)
- added D18: 1N4148, Diode_THT:D_DO-35_SOD27_P7.62mm_Horizontal, B.Cu at (85.5, 99.8)
- added D19: 1N4148, Diode_THT:D_DO-35_SOD27_P7.62mm_Horizontal, B.Cu at (120.0, 129.6)
- added D2: 1N4148, Diode_THT:D_DO-35_SOD27_P7.62mm_Horizontal, B.Cu at (28.5, 87.8)
- added D20: 1N4148, Diode_THT:D_DO-35_SOD27_P7.62mm_Horizontal, B.Cu at (104.5, 61.8)
- added D21: 1N4148, Diode_THT:D_DO-35_SOD27_P7.62mm_Horizontal, B.Cu at (104.5, 80.8)
- added D22: 1N4148, Diode_THT:D_DO-35_SOD27_P7.62mm_Horizontal, B.Cu at (104.5, 99.8)
- added D23: 1N4148, Diode_THT:D_DO-35_SOD27_P7.62mm_Horizontal, B.Cu at (132.6, 144.1)
- added D3: 1N4148, Diode_THT:D_DO-35_SOD27_P7.62mm_Horizontal, B.Cu at (28.5, 106.8)
- added D4: 1N4148, Diode_THT:D_DO-35_SOD27_P7.62mm_Horizontal, B.Cu at (65.7, 120.9)
- added D5: 1N4148, Diode_THT:D_DO-35_SOD27_P7.62mm_Horizontal, B.Cu at (47.5, 37.8)
- added D6: 1N4148, Diode_THT:D_DO-35_SOD27_P7.62mm_Horizontal, B.Cu at (47.5, 56.8)
- added D7: 1N4148, Diode_THT:D_DO-35_SOD27_P7.62mm_Horizontal, B.Cu at (47.5, 75.8)
- added D8: 1N4148, Diode_THT:D_DO-35_SOD27_P7.62mm_Horizontal, B.Cu at (47.5, 94.8)
- added D9: 1N4148, Diode_THT:D_DO-35_SOD27_P7.62mm_Horizontal, B.Cu at (85.3, 120.2)
- added H1: MountingHole, MountingHole:MountingHole_5.3mm_M5_ISO7380, F.Cu at (24.2, 45.5)
- added H10: MountingHole, MountingHole:MountingHole_3.2mm_M3_ISO7380, F.Cu at (71.2, 36.8)
- added H11: MountingHole, MountingHole:MountingHole_3.2mm_M3_ISO7380, F.Cu at (70.2, 121.0)
- added H12: MountingHole, MountingHole:MountingHole_3.2mm_M3_ISO7380, F.Cu at (91.0, 100.8)
- added H13: MountingHole, MountingHole:MountingHole_3.2mm_M3_ISO7380, F.Cu at (132.8, 121.5)
- added H2: MountingHole, MountingHole:MountingHole_5.3mm_M5_ISO7380, F.Cu at (97.8, 38.5)
- added H3: MountingHole, MountingHole:MountingHole_5.3mm_M5_ISO7380, F.Cu at (39.5, 104.0)
- added H4: MountingHole, MountingHole:MountingHole_5.3mm_M5_ISO7380, F.Cu at (122.8, 104.0)
- added H5: MountingHole, MountingHole:MountingHole_3.2mm_M3_ISO7380, F.Cu at (34.8, 57.8)
- added H6: MountingHole, MountingHole:MountingHole_3.2mm_M3_ISO7380, F.Cu at (33.2, 88.8)
- added H7: MountingHole, MountingHole:MountingHole_3.2mm_M3_ISO7380, F.Cu at (71.2, 74.8)
- added H8: MountingHole, MountingHole:MountingHole_3.2mm_M3_ISO7380, F.Cu at (91.0, 62.8)
- added H9: MountingHole, MountingHole:MountingHole_3.2mm_M3_ISO7380, F.Cu at (33.0, 28.0)
- added J1: AudioJack4, Connector_Audio:Jack_3.5mm_PJ320D_Horizontal, F.Cu at (119.5, 82.0)
- added LED1: YS-SK6812MINI-E, kbd:YS-SK6812MINI-E, B.Cu at (24.5, 55.8)
- added LED10: YS-SK6812MINI-E, kbd:YS-SK6812MINI-E, B.Cu at (62.5, 22.8)
- added LED11: YS-SK6812MINI-E, kbd:YS-SK6812MINI-E, B.Cu at (62.5, 41.8)
- added LED12: YS-SK6812MINI-E, kbd:YS-SK6812MINI-E, B.Cu at (62.5, 60.8)
- added LED13: YS-SK6812MINI-E, kbd:YS-SK6812MINI-E, B.Cu at (62.5, 79.8)
- added LED14: YS-SK6812MINI-E, kbd:YS-SK6812MINI-E, B.Cu at (100.5, 105.8)
- added LED15: YS-SK6812MINI-E, kbd:YS-SK6812MINI-E, B.Cu at (81.5, 29.8)
- added LED16: YS-SK6812MINI-E, kbd:YS-SK6812MINI-E, B.Cu at (81.5, 48.8)
- added LED17: YS-SK6812MINI-E, kbd:YS-SK6812MINI-E, B.Cu at (81.5, 67.8)
- added LED18: YS-SK6812MINI-E, kbd:YS-SK6812MINI-E, B.Cu at (81.5, 86.8)
- added LED19: YS-SK6812MINI-E, kbd:YS-SK6812MINI-E, B.Cu at (123.0, 116.4)
- added LED2: YS-SK6812MINI-E, kbd:YS-SK6812MINI-E, B.Cu at (24.5, 74.8)
- added LED20: YS-SK6812MINI-E, kbd:YS-SK6812MINI-E, B.Cu at (100.5, 48.8)
- added LED21: YS-SK6812MINI-E, kbd:YS-SK6812MINI-E, B.Cu at (100.5, 67.8)
- added LED22: YS-SK6812MINI-E, kbd:YS-SK6812MINI-E, B.Cu at (100.5, 86.8)
- added LED23: YS-SK6812MINI-E, kbd:YS-SK6812MINI-E, B.Cu at (139.0, 132.1)
- added LED3: YS-SK6812MINI-E, kbd:YS-SK6812MINI-E, B.Cu at (24.5, 93.8)
- added LED4: YS-SK6812MINI-E, kbd:YS-SK6812MINI-E, B.Cu at (55.8, 111.6)
- added LED5: YS-SK6812MINI-E, kbd:YS-SK6812MINI-E, B.Cu at (43.5, 24.8)
- added LED6: YS-SK6812MINI-E, kbd:YS-SK6812MINI-E, B.Cu at (43.5, 43.8)
- added LED7: YS-SK6812MINI-E, kbd:YS-SK6812MINI-E, B.Cu at (43.5, 62.8)
- added LED8: YS-SK6812MINI-E, kbd:YS-SK6812MINI-E, B.Cu at (43.5, 81.8)
- added LED9: YS-SK6812MINI-E, kbd:YS-SK6812MINI-E, B.Cu at (78.1, 108.7)
- added R1: 10k, Resistor_THT:R_Axial_DIN0207_L6.3mm_D2.5mm_P7.62mm_Horizontal, F.Cu at (119.5, 92.5)
- added R2: 10k, Resistor_THT:R_Axial_DIN0207_L6.3mm_D2.5mm_P7.62mm_Horizontal, F.Cu at (119.5, 89.0)
- added R5: 1k, Resistor_THT:R_Axial_DIN0207_L6.3mm_D2.5mm_P7.62mm_Horizontal, F.Cu at (92.5, 27.8)
- added REF**: KEY_SWITCH, kbd:SW_Hole, F.Cu at (275.5, 254.5)
- added REF**: KEY_SWITCH, kbd:SW_Hole, F.Cu at (237.5, 268.5)
- added REF**: KEY_SWITCH, kbd:SW_Hole, F.Cu at (256.5, 237.5)
- added REF**: KEY_SWITCH, kbd:SW_Hole, F.Cu at (348.8, 305.5)
- added REF**: KEY_SWITCH, kbd:SW_Hole, F.Cu at (294.5, 223.5)
- added REF**: KEY_SWITCH, kbd:SW_Hole, F.Cu at (294.5, 242.5)
- added REF**: KEY_SWITCH, kbd:SW_Hole, F.Cu at (313.5, 280.5)
- added REF**: KEY_SWITCH, kbd:SW_Hole, F.Cu at (313.5, 223.5)
- added REF**: KEY_SWITCH, kbd:SW_Hole, F.Cu at (313.5, 242.5)
- added REF**: KEY_SWITCH, kbd:SW_Hole, F.Cu at (294.5, 204.5)
- added REF**: KEY_SWITCH, kbd:SW_Hole, F.Cu at (256.5, 218.5)
- added REF**: KEY_SWITCH, kbd:SW_Hole, F.Cu at (275.5, 197.5)
- added REF**: KEY_SWITCH, kbd:SW_Hole, F.Cu at (271.0, 285.8)
- added REF**: KEY_SWITCH, kbd:SW_Hole, F.Cu at (237.5, 230.5)
- added REF**: KEY_SWITCH, kbd:SW_Hole, F.Cu at (313.5, 261.5)
- added REF**: KEY_SWITCH, kbd:SW_Hole, F.Cu at (275.5, 235.5)
- added REF**: MountingHole, MountingHole:MountingHole_3.2mm_M3_ISO7380, F.Cu at (246.0, 198.2)
- added REF**: MountingHole, MountingHole:MountingHole_5.3mm_M5_ISO7380, F.Cu at (237.2, 215.8)
- added REF**: MountingHole, MountingHole:MountingHole_5.3mm_M5_ISO7380, F.Cu at (310.8, 208.8)
- added REF**: MountingHole, MountingHole:MountingHole_3.2mm_M3_ISO7380, F.Cu at (345.8, 291.8)
- added REF**: MountingHole, MountingHole:MountingHole_3.2mm_M3_ISO7380, F.Cu at (304.0, 271.0)
- added REF**: MountingHole, MountingHole:MountingHole_3.2mm_M3_ISO7380, F.Cu at (304.0, 233.0)
- added REF**: KEY_SWITCH, kbd:SW_Hole, F.Cu at (256.5, 199.5)
- added REF**: MountingHole, MountingHole:MountingHole_3.2mm_M3_ISO7380, F.Cu at (283.2, 291.2)
- added REF**: MountingHole, MountingHole:MountingHole_5.3mm_M5_ISO7380, F.Cu at (335.8, 274.2)
- added REF**: MountingHole, MountingHole:MountingHole_5.3mm_M5_ISO7380, F.Cu at (252.5, 274.2)
- added REF**: MountingHole, MountingHole:MountingHole_3.2mm_M3_ISO7380, F.Cu at (284.2, 207.0)
- added REF**: MountingHole, MountingHole:MountingHole_3.2mm_M3_ISO7380, F.Cu at (247.8, 228.0)
- added REF**: MountingHole, MountingHole:MountingHole_3.2mm_M3_ISO7380, F.Cu at (246.2, 259.0)
- added REF**: MountingHole, MountingHole:MountingHole_3.2mm_M3_ISO7380, F.Cu at (284.2, 245.0)
- added REF**: MountingHole_3.2mm_M3_ISO7380, MountingHole:MountingHole_3.2mm_M3_ISO7380, F.Cu at (140.8, 284.8)
- added REF**: MountingHole_3.2mm_M3_ISO7380, MountingHole:MountingHole_3.2mm_M3_ISO7380, F.Cu at (99.0, 264.0)
- added REF**: MountingHole_3.2mm_M3_ISO7380, MountingHole:MountingHole_3.2mm_M3_ISO7380, F.Cu at (41.2, 252.0)
- added REF**: KEY_SWITCH, kbd:SW_Hole, F.Cu at (275.5, 216.5)
- added REF**: MountingHole_5.3mm_M5_ISO7380, MountingHole:MountingHole_5.3mm_M5_ISO7380, F.Cu at (32.2, 208.8)
- added REF**: MountingHole_3.2mm_M3_ISO7380, MountingHole:MountingHole_3.2mm_M3_ISO7380, F.Cu at (99.0, 226.0)
- added REF**: MountingHole_3.2mm_M3_ISO7380, MountingHole:MountingHole_3.2mm_M3_ISO7380, F.Cu at (79.2, 200.0)
- added REF**: MountingHole_5.3mm_M5_ISO7380, MountingHole:MountingHole_5.3mm_M5_ISO7380, F.Cu at (105.5, 201.8)
- added REF**: MountingHole_3.2mm_M3_ISO7380, MountingHole:MountingHole_3.2mm_M3_ISO7380, F.Cu at (42.8, 221.0)
- added REF**: MountingHole_3.2mm_M3_ISO7380, MountingHole:MountingHole_3.2mm_M3_ISO7380, F.Cu at (79.2, 238.0)
- added REF**: MountingHole_3.2mm_M3_ISO7380, MountingHole:MountingHole_3.2mm_M3_ISO7380, F.Cu at (78.2, 284.2)
- added REF**: MountingHole_5.3mm_M5_ISO7380, MountingHole:MountingHole_5.3mm_M5_ISO7380, F.Cu at (47.5, 267.2)
- added REF**: MountingHole_3.2mm_M3_ISO7380, MountingHole:MountingHole_3.2mm_M3_ISO7380, F.Cu at (41.0, 191.2)
- added REF**: MountingHole_5.3mm_M5_ISO7380, MountingHole:MountingHole_5.3mm_M5_ISO7380, F.Cu at (130.8, 267.2)
- added REF**: KEY_SWITCH, kbd:SW_Hole, F.Cu at (256.5, 256.5)
- added REF**: KEY_SWITCH, kbd:SW_Hole, F.Cu at (294.5, 261.5)
- added REF**: KEY_SWITCH, kbd:SW_Hole, F.Cu at (333.8, 290.5)
- added REF**: KEY_SWITCH, kbd:SW_Hole, F.Cu at (292.2, 283.2)
- added REF**: KEY_SWITCH, kbd:SW_Hole, F.Cu at (237.5, 249.5)
- added SW1: SW_Push, kbd:CherryMX_Hotswap, F.Cu at (24.5, 60.2)
- added SW10: SW_Push, kbd:CherryMX_Hotswap, F.Cu at (62.5, 27.2)
- added SW11: SW_Push, kbd:CherryMX_Hotswap, F.Cu at (62.5, 46.2)
- added SW12: SW_Push, kbd:CherryMX_Hotswap, F.Cu at (62.5, 65.2)
- added SW13: SW_Push, kbd:CherryMX_Hotswap, F.Cu at (62.5, 84.2)
- added SW14: SW_Push, kbd:CherryMX_Hotswap, F.Cu at (100.5, 110.2)
- added SW15: SW_Push, kbd:CherryMX_Hotswap, F.Cu at (81.5, 34.2)
- added SW16: SW_Push, kbd:CherryMX_Hotswap, F.Cu at (81.5, 53.2)
- added SW17: SW_Push, kbd:CherryMX_Hotswap, F.Cu at (81.5, 72.2)
- added SW18: SW_Push, kbd:CherryMX_Hotswap, F.Cu at (81.5, 91.2)
- added SW19: SW_Push, kbd:CherryMX_Hotswap, F.Cu at (120.8, 120.2)
- added SW2: SW_Push, kbd:CherryMX_Hotswap, F.Cu at (24.5, 79.2)
- added SW20: SW_Push, kbd:CherryMX_Hotswap, F.Cu at (100.5, 53.2)
- added SW21: SW_Push, kbd:CherryMX_Hotswap, F.Cu at (100.5, 72.2)
- added SW22: SW_Push, kbd:CherryMX_Hotswap, F.Cu at (100.5, 91.2)
- added SW23: SW_Push, kbd:CherryMX_Hotswap, F.Cu at (135.8, 135.2)
- added SW3: SW_Push, kbd:CherryMX_Hotswap, F.Cu at (24.5, 98.2)
- added SW4: SW_Push, kbd:CherryMX_Hotswap, F.Cu at (58.0, 115.5)
- added SW47: SW_Push, Button_Switch_THT:SW_PUSH_6mm_H7.3mm, F.Cu at (112.0, 95.5)
- added SW5: SW_Push, kbd:CherryMX_Hotswap, F.Cu at (43.5, 29.2)
- added SW6: SW_Push, kbd:CherryMX_Hotswap, F.Cu at (43.5, 48.2)
- added SW7: SW_Push, kbd:CherryMX_Hotswap, F.Cu at (43.5, 67.2)
- added SW8: SW_Push, kbd:CherryMX_Hotswap, F.Cu at (43.5, 86.2)
- added SW9: SW_Push, kbd:CherryMX_Hotswap, F.Cu at (79.2, 113.0)
- added U1: ProMicro, kbd:ProMicro_v3.5, F.Cu at (119.2, 62.0)
- moved D46 176.8 mm to (283.7, 127.1)
- moved C24 176.8 mm to (244.5, 47.5)
- moved C25 176.8 mm to (244.5, 66.5)
- moved C26 176.8 mm to (244.0, 85.5)
- moved C27 176.8 mm to (202.5, 130.4)
- moved C28 176.8 mm to (263.5, 28.4)
- moved C29 176.8 mm to (263.0, 47.5)
- moved C30 176.8 mm to (263.0, 67.0)
- moved C31 176.8 mm to (263.0, 85.5)
- moved C32 176.8 mm to (219.5, 114.6)
- moved C33 176.8 mm to (282.0, 21.5)
- moved C34 176.8 mm to (282.0, 40.5)
- moved C35 176.8 mm to (281.5, 60.0)
- moved C36 176.8 mm to (281.5, 78.5)
- moved C37 176.8 mm to (243.5, 104.5)
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Connections:
- LED25 pad 4: Net-(LED24-Pad4) -> Net-(LED25-Pad4)
- LED27 pad 4: Net-(LED26-Pad4) -> Net-(LED27-Pad4)
- LED38 pad 2: Net-(LED38-Pad2) -> Net-(LED24-Pad4)
- LED43 pad 2: Net-(LED38-Pad2) -> Net-(LED25-Pad4)
- LED44 pad 2: Net-(LED44-Pad2) -> Net-(LED26-Pad4)
- LED45 pad 2: Net-(LED44-Pad2) -> Net-(LED27-Pad4)
Routing:
- net +5V: track 904.2 -> 1689.4 mm
- net GND: track 662.2 -> 1324.7 mm, vias 0 -> 1
- net /lcol1: track 0.00 -> 193.7 mm, vias 0 -> 6
- net /lcol0: track 0.00 -> 182.6 mm, vias 0 -> 3
- net /lcol3: track 0.00 -> 167.5 mm, vias 0 -> 3
- net /lcol2: track 0.00 -> 166.8 mm, vias 0 -> 3
- net /lcol4: track 0.00 -> 138.4 mm, vias 0 -> 2
- net /lrow4: track 0.00 -> 134.9 mm, vias 0 -> 2
- net /lrow3: track 0.00 -> 124.7 mm, vias 0 -> 1
- net /lrow2: track 0.00 -> 106.6 mm
- net /lrow1: track 0.00 -> 93.4 mm
- net /lrow0: track 0.00 -> 78.5 mm
- net Net-(LED22-Pad2): track 0.00 -> 70.6 mm, vias 0 -> 2
- net /lRST: track 0.00 -> 45.3 mm
- net Net-(LED1-Pad4): track 0.00 -> 42.0 mm, vias 0 -> 2
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Other:
- board size 134.1 x 130.9 mm -> 347.1 x 301.1 mm

Commit message: Update
Parts:
- removed C1, C10, C11, C12, C13, C14, C15, C16, C17, C18, C19, C2, C20, C21, C22, C23, C3, C4, C5, C6, C7, C8, C9: 0.1uF, Capacitor_THT:C_Disc_D6.0mm_W2.5mm_P5.00mm
- removed D1, D10, D11, D12, D13, D14, D15, D16, D17, D18, D19, D2, D20, D21, D22, D23, D3, D4, D5, D6, D7, D8, D9: 1N4148, Diode_THT:D_DO-35_SOD27_P7.62mm_Horizontal
- removed H1, H2, H3, H4, REF** (x4): MountingHole, MountingHole:MountingHole_5.3mm_M5_ISO7380
- removed H10, H11, H12, H13, H5, H6, H7, H8, H9, REF** (x9): MountingHole, MountingHole:MountingHole_3.2mm_M3_ISO7380
- removed J1: AudioJack4, Connector_Audio:Jack_3.5mm_PJ320D_Horizontal
- removed LED1, LED10, LED11, LED12, LED13, LED14, LED15, LED16, LED17, LED18, LED19, LED2, LED20, LED21, LED22, LED23, LED3, LED4, LED5, LED6, LED7, LED8, LED9: YS-SK6812MINI-E, kbd:YS-SK6812MINI-E
- removed R1, R2: 10k, Resistor_THT:R_Axial_DIN0207_L6.3mm_D2.5mm_P7.62mm_Horizontal
- removed R5: 1k, Resistor_THT:R_Axial_DIN0207_L6.3mm_D2.5mm_P7.62mm_Horizontal
- removed REF** (x23): KEY_SWITCH, kbd:SW_Hole
- removed REF** (x9): MountingHole_3.2mm_M3_ISO7380, MountingHole:MountingHole_3.2mm_M3_ISO7380
- removed REF** (x4): MountingHole_5.3mm_M5_ISO7380, MountingHole:MountingHole_5.3mm_M5_ISO7380
- removed SW1, SW10, SW11, SW12, SW13, SW14, SW15, SW16, SW17, SW18, SW19, SW2, SW20, SW21, SW22, SW23, SW3, SW4, SW5, SW6, SW7, SW8, SW9: SW_Push, kbd:CherryMX_Hotswap
- removed SW47: SW_Push, Button_Switch_THT:SW_PUSH_6mm_H7.3mm
- removed U1: ProMicro, kbd:ProMicro_v3.5
- moved C46 192.6 mm to (98.3, 94.9)
- moved D42 192.6 mm to (73.0, 107.6)
- moved D46 192.6 mm to (91.8, 110.2)
- moved LED42 192.6 mm to (72.5, 94.0)
- moved C24 192.6 mm to (52.6, 30.6)
- moved C25 192.6 mm to (52.6, 49.6)
- moved C26 192.6 mm to (52.1, 68.6)
- moved C28 192.6 mm to (71.6, 11.6)
- moved C29 192.6 mm to (71.1, 30.6)
- moved C30 192.6 mm to (71.1, 50.1)
- moved C31 192.6 mm to (71.1, 68.6)
- moved C32 192.6 mm to (27.6, 97.7)
- moved C33 192.6 mm to (90.1, 4.61)
- moved C34 192.6 mm to (90.1, 23.6)
- moved C35 192.6 mm to (89.6, 43.1)
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Routing:
- net +5V: track 1689.4 -> 904.2 mm
- net GND: track 1324.7 -> 662.2 mm, vias 1 -> 0
- net /lcol1: track 193.7 -> 0.00 mm, vias 6 -> 0
- net /lcol0: track 182.6 -> 0.00 mm, vias 3 -> 0
- net /lcol3: track 167.5 -> 0.00 mm, vias 3 -> 0
- net /lcol2: track 166.8 -> 0.00 mm, vias 3 -> 0
- net /lcol4: track 138.4 -> 0.00 mm, vias 2 -> 0
- net /lrow4: track 134.9 -> 0.00 mm, vias 2 -> 0
- net /lrow3: track 124.7 -> 0.00 mm, vias 1 -> 0
- net /lrow2: track 106.6 -> 0.00 mm
- net /lrow1: track 93.4 -> 0.00 mm
- net /lrow0: track 78.5 -> 0.00 mm
- net Net-(LED22-Pad2): track 70.6 -> 0.00 mm, vias 2 -> 0
- net /lRST: track 45.3 -> 0.00 mm
- net Net-(LED1-Pad4): track 42.0 -> 0.00 mm, vias 2 -> 0
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Other:
- board size 347.1 x 301.1 mm -> 134.1 x 130.9 mm
- net class Default removed
- net class Power removed

Commit message: Update
Parts:
- moved R6 4.73 mm to (61.1, 16.8)
- moved C46 4.63 mm to (101.4, 98.4)
- moved C30 4.63 mm to (74.1, 53.6)
- moved C35 4.63 mm to (92.6, 46.6)
- moved C36 4.63 mm to (92.6, 65.1)
- moved C40 4.63 mm to (112.1, 48.1)
- moved C41 4.63 mm to (112.1, 67.1)
- moved D29 4.63 mm to (76.1, 50.6)
- moved D34 4.63 mm to (95.1, 43.6)
- moved D35 4.63 mm to (95.1, 62.6)
- moved D39 4.63 mm to (114.1, 45.6)
- moved D40 4.63 mm to (114.1, 64.6)
- moved H19 4.63 mm to (118.9, 46.6)
- moved H22 4.63 mm to (82.4, 63.6)
- moved LED29 4.63 mm to (72.1, 37.6)
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Routing:
- net Net-(LED27-Pad4): track 0.00 -> 161.8 mm, vias 0 -> 2
- net Net-(LED25-Pad4): track 0.00 -> 96.5 mm, vias 0 -> 2
- net Net-(LED24-Pad4): track 22.7 -> 81.6 mm
- net Net-(LED38-Pad2): track 40.6 -> 0.00 mm, vias 2 -> 0
- net Net-(LED44-Pad2): track 39.0 -> 0.00 mm
- net /rLED: track 25.5 -> 0.00 mm
- net Net-(LED26-Pad4): track 73.3 -> 94.2 mm
- net Net-(LED28-Pad4): track 9.37 -> 0.00 mm
- net +5V: track 904.2 -> 897.8 mm
- net /rrow4: track 157.1 -> 151.2 mm, vias 2 -> 3
- net /rcol3: track 200.0 -> 202.9 mm, vias 5 -> 9
- net GND: track 662.2 -> 663.2 mm
- net /rcol2: track 181.4 -> 182.5 mm, vias 4 -> 8
- net /rrow1: track 124.8 -> 125.5 mm
- net /rcol1: track 169.2 -> 169.9 mm, vias 5 -> 9
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Other:
- rule pad_to_mask_clearance: 0.05 -> 0
