File: pcb/right.kicad_pcb (KiCad board)
At the start: 2 copper layers, 123.5 x 102 mm, 110 parts, among them J2 USB_B_Micro, SW24 SW_Push, SW25 SW_Push, SW26 SW_Push, SW27 SW_Push, SW28 SW_Push, SW29 SW_Push, SW30 SW_Push, SW31 SW_Push, SW32 SW_Push, SW33 SW_Push, SW34 SW_Push, SW35 SW_Push, SW36 SW_Push, SW37 SW_Push, SW38 SW_Push, SW39 SW_Push, SW40 SW_Push, SW41 SW_Push, SW42 SW_Push, SW43 SW_Push, SW44 SW_Push, SW45 SW_Push, SW46 SW_Push, SW48 SW_Push, SW50 SW_Push, U2 ProMicro

Commit message: update
Routing:
- net +5V: track 0.00 -> 674.0 mm
- net GND: track 0.00 -> 645.3 mm
- net /rcol2: track 0.00 -> 211.8 mm, vias 0 -> 1
- net /rcol4: track 0.00 -> 209.4 mm, vias 0 -> 1
- net /rcol3: track 0.00 -> 209.3 mm, vias 0 -> 1
- net /rcol1: track 0.00 -> 190.3 mm, vias 0 -> 2
- net /rcol0: track 0.00 -> 174.7 mm
- net /rrow4: track 0.00 -> 155.3 mm
- net /rrow3: track 0.00 -> 124.0 mm
- net /rrow2: track 0.00 -> 116.8 mm
- net Net-(LED27-Pad4): track 0.00 -> 116.2 mm, vias 0 -> 2
- net /rrow0: track 0.00 -> 115.1 mm
- net /rrow1: track 0.00 -> 111.7 mm
- net Net-(LED25-Pad4): track 0.00 -> 89.5 mm, vias 0 -> 2
- net Net-(LED26-Pad4): track 0.00 -> 80.3 mm, vias 0 -> 2
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