File: choc/memekbd.kicad_pcb (KiCad board)
At the start: 2 copper layers, 277.2 x 195.2 mm, 212 parts, among them J1 USB_B_Micro, J2 USB_B_Micro, SW1 SW_Push, SW10 SW_Push, SW11 SW_Push, SW12 SW_Push, SW13 SW_Push, SW14 SW_Push, SW15 SW_Push, SW16 SW_Push, SW17 SW_Push, SW18 SW_Push, SW19 SW_Push, SW2 SW_Push, SW20 SW_Push, SW21 SW_Push, SW22 SW_Push, SW23 SW_Push, SW24 SW_Push, SW25 SW_Push, SW26 SW_Push, SW27 SW_Push, SW28 SW_Push, SW29 SW_Push, SW3 SW_Push, SW30 SW_Push, SW31 SW_Push, SW32 SW_Push, SW33 SW_Push, SW34 SW_Push, SW35 SW_Push, SW36 SW_Push, SW37 SW_Push, SW38 SW_Push, SW39 SW_Push, SW4 SW_Push, SW40 SW_Push, SW41 SW_Push, SW42 SW_Push, SW43 SW_Push, SW44 SW_Push, SW45 SW_Push, SW46 SW_Push, SW47 SW_Push, SW48 SW_Push, SW49 SW_Push, SW5 SW_Push, SW50 SW_Push, SW6 SW_Push, SW7 SW_Push, SW8 SW_Push, SW9 SW_Push, U1 ProMicro, U2 ProMicro

Commit message: remove leds from choc
Parts:
- removed LED1, LED10, LED11, LED12, LED13, LED14, LED15, LED16, LED17, LED18, LED19, LED2, LED20, LED21, LED22, LED23, LED24, LED25, LED26, LED27, LED28, LED29, LED3, LED30, LED31, LED32, LED33, LED34, LED35, LED36, LED37, LED38, LED39, LED4, LED40, LED41, LED42, LED43, LED44, LED45, LED46, LED47, LED48, LED5, LED6, LED7, LED8, LED9: YS-SK6812MINI-E, kbd:YS-SK6812MINI-E
- removed R5, R6: 1k, Resistor_THT:R_Axial_DIN0207_L6.3mm_D2.5mm_P7.62mm_Horizontal
- removed the REF** at (185.2, 198.8)
- removed the REF** at (185.2, 171.8)
- removed the REF** at (78.5, 199.2)
- removed the REF** at (185.2, 154.8)
- removed the REF** at (257.2, 130.8)
- removed the REF** at (256.8, 119.0)
- removed the REF** at (203.2, 181.8)
- removed the REF** at (117.0, 199.2)
- removed the REF** at (257.2, 181.8)
- removed the REF** at (233.5, 119.0)
- removed the REF** at (185.2, 137.8)
- removed the REF** at (215.5, 186.8)
- removed the REF** at (78.5, 124.8)
- removed the REF** at (181.0, 120.0)
- removed the REF** at (24.5, 191.0)
- removed the REF** at (203.2, 159.8)
- removed the REF** at (233.5, 193.5)
- removed the REF** at (179.5, 185.2)
- removed the REF** at (275.2, 181.8)
- removed the REF** at (272.0, 193.5)
- removed the REF** at (26.0, 125.8)
- removed the REF** at (284.2, 198.8)
- removed the REF** at (257.2, 147.8)
- removed the REF** at (203.2, 142.8)
- removed the REF** at (221.2, 140.8)
- removed the REF** at (203.2, 125.8)
- removed the REF** at (203.2, 198.8)
- removed the REF** at (239.2, 130.8)
- removed the REF** at (101.8, 124.8)
- removed the REF** at (257.2, 164.8)
- removed the REF** at (221.2, 198.8)
- removed the REF** at (221.2, 174.8)
- removed the REF** at (239.2, 164.8)
- removed the REF** at (60.5, 192.5)
- removed the REF** at (239.2, 181.8)
- removed the REF** at (221.2, 123.8)
- removed the REF** at (221.2, 157.8)
- removed the REF** at (239.2, 147.8)
- added REF**: MountingHole_Pad, MountingHole:MountingHole_3.2mm_M3_ISO7380_Pad, F.Cu at (216.0, 191.0)
- added REF**: KEY_SWITCH, kbd:ChocV1_Hole, F.Cu at (221.8, 203.0)
- added REF**: KEY_SWITCH, kbd:ChocV1_Hole, F.Cu at (257.8, 186.0)
- added REF**: KEY_SWITCH, kbd:ChocV1_Hole, F.Cu at (185.8, 142.0)
- added REF**: KEY_SWITCH, kbd:ChocV1_Hole, F.Cu at (284.8, 203.0)
- added REF**: KEY_SWITCH, kbd:ChocV1_Hole, F.Cu at (239.8, 186.0)
- added REF**: KEY_SWITCH, kbd:ChocV1_Hole, F.Cu at (257.8, 135.0)
- added REF**: KEY_SWITCH, kbd:ChocV1_Hole, F.Cu at (221.8, 145.0)
- added REF**: KEY_SWITCH, kbd:ChocV1_Hole, F.Cu at (203.8, 147.0)
- added REF**: KEY_SWITCH, kbd:ChocV1_Hole, F.Cu at (257.8, 169.0)
- added REF**: KEY_SWITCH, kbd:ChocV1_Hole, F.Cu at (239.8, 135.0)
- added REF**: MountingHole_Pad, MountingHole:MountingHole_3.2mm_M3_ISO7380_Pad, F.Cu at (61.0, 196.8)
- added REF**: MountingHole_Pad, MountingHole:MountingHole_3.2mm_M3_ISO7380_Pad, F.Cu at (180.0, 189.5)
- added REF**: MountingHole_Pad, MountingHole:MountingHole_3.2mm_M3_ISO7380_Pad, F.Cu at (25.0, 195.2)
- added REF**: MountingHole_Pad, MountingHole:MountingHole_3.2mm_M3_ISO7380_Pad, F.Cu at (234.0, 197.8)
- added REF**: KEY_SWITCH, kbd:ChocV1_Hole, F.Cu at (275.8, 186.0)
- added REF**: MountingHole_Pad, MountingHole:MountingHole_3.2mm_M3_ISO7380_Pad, F.Cu at (102.2, 129.0)
- added REF**: KEY_SWITCH, kbd:ChocV1_Hole, F.Cu at (257.8, 152.0)
- added REF**: KEY_SWITCH, kbd:ChocV1_Hole, F.Cu at (239.8, 169.0)
- added REF**: KEY_SWITCH, kbd:ChocV1_Hole, F.Cu at (239.8, 152.0)
- added REF**: MountingHole_Pad, MountingHole:MountingHole_3.2mm_M3_ISO7380_Pad, F.Cu at (181.5, 124.2)
- added REF**: KEY_SWITCH, kbd:ChocV1_Hole, F.Cu at (185.8, 159.0)
- added REF**: KEY_SWITCH, kbd:ChocV1_Hole, F.Cu at (203.8, 164.0)
- added REF**: MountingHole_Pad, MountingHole:MountingHole_3.2mm_M3_ISO7380_Pad, F.Cu at (26.5, 130.0)
- added REF**: KEY_SWITCH, kbd:ChocV1_Hole, F.Cu at (203.8, 130.0)
- added REF**: KEY_SWITCH, kbd:ChocV1_Hole, F.Cu at (203.8, 203.0)
- added REF**: MountingHole_Pad, MountingHole:MountingHole_3.2mm_M3_ISO7380_Pad, F.Cu at (272.5, 197.8)
- added REF**: MountingHole_Pad, MountingHole:MountingHole_3.2mm_M3_ISO7380_Pad, F.Cu at (257.2, 123.2)
- added REF**: KEY_SWITCH, kbd:ChocV1_Hole, F.Cu at (221.8, 128.0)
- added REF**: MountingHole_Pad, MountingHole:MountingHole_3.2mm_M3_ISO7380_Pad, F.Cu at (79.0, 129.0)
- added REF**: KEY_SWITCH, kbd:ChocV1_Hole, F.Cu at (185.8, 203.0)
- added REF**: KEY_SWITCH, kbd:ChocV1_Hole, F.Cu at (185.8, 176.0)
- added REF**: KEY_SWITCH, kbd:ChocV1_Hole, F.Cu at (221.8, 179.0)
- added REF**: MountingHole_Pad, MountingHole:MountingHole_3.2mm_M3_ISO7380_Pad, F.Cu at (79.0, 203.5)
- added REF**: KEY_SWITCH, kbd:ChocV1_Hole, F.Cu at (221.8, 162.0)
- added REF**: MountingHole_Pad, MountingHole:MountingHole_3.2mm_M3_ISO7380_Pad, F.Cu at (234.0, 123.2)
- added REF**: MountingHole_Pad, MountingHole:MountingHole_3.2mm_M3_ISO7380_Pad, F.Cu at (117.5, 203.5)
- added REF**: KEY_SWITCH, kbd:ChocV1_Hole, F.Cu at (203.8, 186.0)
Other:
- board size 277.2 x 195.2 mm -> 277.8 x 199.5 mm
